File: board/HyperFusionXC.kicad_pcb (KiCad board)
At the start: 2 copper layers, 99 x 65.6 mm, 103 parts, among them J1 Conn_01x02_Pin, U1 10CL025YE144C8G, U10 SN74LVC1G04DCKR, U12 TXS0108EPWR, U14 TXS0108EPWR, U2 74AHC541, U3 74AHC541, U4 M25P80-VMN3TPB, U5 PCM5101APWR, U6 AT93C46DN-SH-T, U7 SG3225CAN 50.0000M-TJGA6, U8 74AHC541, U9 PCM1808PWR, X1 EDGE50/MSX, X3 302-S101

Commit message: Work in progress
Parts:
- added C16: 100nF, Capacitor_SMD:C_0603_1608Metric, F.Cu at (135.2, 119.1)
- added C17: 100nF, Capacitor_SMD:C_0603_1608Metric, F.Cu at (145.2, 119.1)
- added C45: 100nF, Capacitor_SMD:C_0603_1608Metric, F.Cu at (160.2, 118.8)
- U7: moved to F.Cu
- moved U7 38.8 mm to (129.4, 107.2), turned to 0 degrees
- moved U1 5.71 mm to (144.8, 101.7)
- moved U8 2.93 mm to (150.5, 118.9)
- moved U2 2.88 mm to (150.5, 118.9)
- moved U3 2.58 mm to (140.0, 118.9)
- moved U12 2.58 mm to (140.0, 118.9)
- moved U10 2.48 mm to (156.5, 116.7), turned to 0 degrees
Connections:
- net /~{SLT_SW} renamed /~{SLT_MUX}
- U1 pad 22: /SLT_CLC -> GND
- U1 pad 58: /SLT_Y3 -> /SLT_MUX
- U1 pad 59: /SLT_Y2 -> /SLT_Y0
- U1 pad 60: /SLT_Y1 -> /SLT_Y2
- U1 pad 65: /SLT_Y0 -> /SLT_Y1
- U1 pad 66: /SLT_SW -> /SLT_Y3
- U1 pad 67: /~{SLT_SLTSL} -> /~{SLT_RFSH}
- U1 pad 68: /~{SLT_RFSH} -> /~{SLT_WAIT}
- U1 pad 69: /~{SLT_WAIT} -> /~{SLT_RESET}
- U1 pad 71: /~{SLT_INT} -> /~{SLT_BUSDIR}
- U1 pad 72: /~{SLT_BUSDIR} -> /~{SLT_INT}
- U1 pad 76: /~{SLT_RESET} -> /~{SLT_SLTSL}
- U1 pad 88: GND -> /SLT_CLC
- U10 pad 2: /SLT_SW -> /SLT_MUX
- U10 pad 3: unconnected-(U10-GND-Pad3) -> GND
- U10 pad 5: unconnected-(U10-VCC-Pad5) -> +3V3
- U12 pad 10: /SLT_SW -> /SLT_MUX
- U14 pad 1: /~{SLT_SLTSL} -> unconnected-(U14-A1-Pad1)
- U14 pad 12: /EDGE_CLC -> /~{EDGE_RESET}
- U14 pad 13: unconnected-(U14-B7-Pad13) -> /~{EDGE_BUSDIR}
- U14 pad 14: /~{EDGE_RESET} -> /~{EDGE_INT}
- U14 pad 15: /~{EDGE_BUSDIR} -> /~{EDGE_WAIT}
- U14 pad 16: /~{EDGE_INT} -> /~{EDGE_RFSH}
- U14 pad 17: /~{EDGE_WAIT} -> /~{EDGE_SLTSEL}
- U14 pad 18: /~{EDGE_RFSH} -> /EDGE_CLC
- U14 pad 20: /~{EDGE_SLTSEL} -> unconnected-(U14-B1-Pad20)
- U14 pad 3: /~{SLT_RFSH} -> /SLT_CLC
- U14 pad 4: /~{SLT_WAIT} -> /~{SLT_SLTSL}
- U14 pad 5: /~{SLT_INT} -> /~{SLT_RFSH}
- U14 pad 6: /~{SLT_BUSDIR} -> /~{SLT_WAIT}
- U14 pad 7: /~{SLT_RESET} -> /~{SLT_INT}
- U14 pad 8: unconnected-(U14-A7-Pad8) -> /~{SLT_BUSDIR}
- U14 pad 9: /SLT_CLC -> /~{SLT_RESET}
- U3 pad 1: /SLT_SW -> /SLT_MUX
- U3 pad 11: /SLT_X7 -> /SLT_X6
- U3 pad 12: /SLT_X6 -> /SLT_X7
- U3 pad 13: /SLT_X5 -> /SLT_X4
- U3 pad 14: /SLT_X4 -> /SLT_X5
- U3 pad 15: /SLT_X3 -> /SLT_X2
- U3 pad 16: /SLT_X2 -> /SLT_X3
- U3 pad 17: /SLT_X1 -> /SLT_X0
- U3 pad 18: /SLT_X0 -> /SLT_X1
- U3 pad 19: /SLT_SW -> /SLT_MUX
- U3 pad 2: /EDGE_A6 -> /EDGE_A7
- U3 pad 3: /EDGE_A7 -> /EDGE_A6
- U3 pad 4: /EDGE_A0 -> /EDGE_A1
- U3 pad 5: /EDGE_A1 -> /EDGE_A0
- U3 pad 6: /EDGE_A2 -> /EDGE_A3
- U3 pad 7: /EDGE_A3 -> /EDGE_A2
- U3 pad 8: /EDGE_A4 -> /EDGE_A5
- U3 pad 9: /EDGE_A5 -> /EDGE_A4
- U8 pad 1: /SLT_SW -> /SLT_MUX
- U8 pad 19: /SLT_SW -> /SLT_MUX
- U8 pad 2: /~{EDGE_CS1} -> /~{EDGE_CS2}
- U8 pad 3: /~{EDGE_CS2} -> /~{EDGE_CS1}
Routing:
- net +5V: track 0.00 -> 74.8 mm, vias 0 -> 3
- net GND: track 0.00 -> 72.1 mm, vias 0 -> 4
- net +3V3: track 18.8 -> 83.2 mm, vias 1 -> 6
- net /SLT_MUX: track 0.00 -> 63.2 mm, vias 0 -> 5
- net /~{EDGE_WR}: track 0.00 -> 23.7 mm
- net /~{SLT_MUX}: track 0.00 -> 20.4 mm, vias 0 -> 2
- net /SLT_Y5: track 0.00 -> 18.5 mm, vias 0 -> 1
- net /SLT_Y4: track 0.00 -> 18.4 mm, vias 0 -> 1
- net /~{SLT_RFSH}: track 0.00 -> 18.2 mm
- net /SLT_CLC: track 0.00 -> 18.1 mm
- net /SLT_Y0: track 0.00 -> 17.2 mm, vias 0 -> 2
- net /~{SLT_WAIT}: track 0.00 -> 16.5 mm
- net /~{SLT_SLTSL}: track 0.00 -> 13.6 mm
- net /SLT_Y2: track 0.00 -> 13.4 mm, vias 0 -> 2
- net /~{SLT_RESET}: track 0.00 -> 12.8 mm
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
Commit message: Work in progress
Parts:
- moved U7 43.4 mm to (86.0, 108.5)
- turned R57 to 90 degrees
Connections:
- U1 pad 10: /DAC_LRCK -> /DAC_DIN
- U1 pad 11: /DAC_DIN -> /DAC_BCK
- U1 pad 136: /ADC_MD1 -> unconnected-(U1-IO_56-Pad136)
- U1 pad 137: /ADC_MD0 -> unconnected-(U1-IO_57-Pad137)
- U1 pad 141: /ADC_DOUT -> /ADC_BCK
- U1 pad 142: /ADC_BCK -> /ADC_LRCK
- U1 pad 144: /ADC_LRCK -> /DAC_XSMT
- U1 pad 15: unconnected-(U1-TDI-Pad15) -> /TDI
- U1 pad 16: unconnected-(U1-TCK-Pad16) -> /TCK
- U1 pad 18: unconnected-(U1-TMS-Pad18) -> /TMS
- U1 pad 20: unconnected-(U1-TDO-Pad20) -> /TDO
- U1 pad 22: GND -> /ADC_DOUT
- U1 pad 28: /DAC_BCK -> /DAC_SCK
- U1 pad 31: /DAC_SCK -> /DAC_BCK
- U1 pad 32: /DAC_FLT -> /DAC_SCK
- U1 pad 33: /DAC_DEMP -> /DAC_FLT
- U1 pad 7: /DAC_XSMT -> /DAC_LRCK
- U5 pad 10: /DAC_DEMP -> GND
- U9 pad 10: /ADC_MD0 -> GND
- U9 pad 11: /ADC_MD1 -> GND
Routing:
- net GND: track 72.1 -> 279.1 mm, vias 4 -> 8
- net +3V3: track 83.2 -> 179.2 mm, vias 6 -> 12
- net +5V: track 74.8 -> 159.7 mm, vias 3 -> 10
- net /TDO: track 0.00 -> 47.4 mm
- net /TMS: track 2.61 -> 45.5 mm
- net /TDI: track 4.20 -> 44.0 mm, vias 0 -> 1
- net /TCK: track 14.1 -> 51.9 mm
- net /ADC_DOUT: track 0.00 -> 23.9 mm, vias 0 -> 2
- net +1V2: track 0.00 -> 20.0 mm, vias 0 -> 1
- net /DAC_XSMT: track 0.00 -> 18.8 mm, vias 0 -> 2
- net /ADC_LRCK: track 0.00 -> 18.3 mm, vias 0 -> 2
- net /ADC_SCKI: track 0.00 -> 16.6 mm, vias 0 -> 2
- net /DAC_LRCK: track 0.00 -> 14.2 mm, vias 0 -> 2
- net /DAC_BCK: track 0.00 -> 13.7 mm
- net /DAC_DIN: track 0.00 -> 13.6 mm, vias 0 -> 2
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- removed copper zone on F.Cu, net +1V2
- removed copper zone on F.Cu, net +3.3VDAC
- removed copper zone on F.Cu, net +3V3
- removed copper zone on B.Cu, net /TCK
- removed copper zone on F.Cu, net /TCK
- removed copper zone on B.Cu, net GND
- removed copper zone on F.Cu, net GND
- removed copper zone on B.Cu, net GNDA
- removed copper zone on F.Cu, net GNDA
Other:
- board text added: "AX1"
- board text added: "AX2"
- board text removed: "HyperFusionXC v1.0 MSX Cartridge SHS 2025"
- board text removed: "JTAG"
- board text removed: "Line-Out"

Commit message: Work in progress
Parts:
- removed C39, C40, C41, C42, C43: 100nF, Capacitor_SMD:C_0603_1608Metric
- removed R43, R44, R63, R65, R66, R67, R68, R69: 10E, Resistor_SMD:R_0603_1608Metric
- removed R46, R47, R48, R56, R58, R59: 10k, Resistor_SMD:R_0603_1608Metric
- removed R49, R60, R61: 470E, Resistor_SMD:R_0603_1608Metric
- removed R57, R70, R71: 1k, Resistor_SMD:R_0603_1608Metric
- removed R62: 25E, Resistor_SMD:R_0603_1608Metric
- removed TP1: TestPoint, Library:TestPoint_THTPad_D1.5mm_Drill0.9mm
- removed U7: SG3225CAN 50.0000M-TJGA6, Library:SG3225CAN
- removed UCT1: AP2114HA-1.2TRG1, Package_TO_SOT_SMD:SOT-223
- removed UCT2, UCT3: AP2111H-3.3TRG1, Package_TO_SOT_SMD:SOT-223
- added AX3: SJ1-3523N, Library:ST-222_1, F.Cu at (189.6, 76.0)
- added C4: 100nF, Capacitor_SMD:C_0603_1608Metric, F.Cu at (169.3, 101.8)
- added C5: 100nF, Capacitor_SMD:C_0603_1608Metric, F.Cu at (171.1, 101.8)
- added J2: 10067847-001RLF, Library:AMPHENOL_10067847-001RLF, B.Cu at (141.2, 75.0)
- added MP1: M2.5 x 1.5mm, Library:WA-SMSI_9774015151, F.Cu at (161.3, 84.9)
- added R1: 10k, Resistor_SMD:R_0603_1608Metric, F.Cu at (171.1, 116.4)
- added R10: 100E, Resistor_SMD:R_0603_1608Metric, F.Cu at (182.0, 96.3)
- added R11: 10k, Resistor_SMD:R_0603_1608Metric, F.Cu at (183.8, 115.0)
- added R13: 300k, Resistor_SMD:R_0603_1608Metric, F.Cu at (129.4, 111.4)
- added R14: 200E, Resistor_SMD:R_0603_1608Metric, F.Cu at (79.9, 108.1)
- added R15: 200E, Resistor_SMD:R_0603_1608Metric, F.Cu at (79.9, 110.6)
- added R16: 200E, Resistor_SMD:R_0603_1608Metric, F.Cu at (79.9, 113.1)
- added R17: 200E, Resistor_SMD:R_0603_1608Metric, F.Cu at (83.9, 100.5)
- added R18: 200E, Resistor_SMD:R_0603_1608Metric, F.Cu at (83.9, 103.0)
- added R19: 200E, Resistor_SMD:R_0603_1608Metric, F.Cu at (83.9, 105.5)
- added R2: 10k, Resistor_SMD:R_0603_1608Metric, F.Cu at (171.1, 118.9)
- added R20: 100E, Resistor_SMD:R_0603_1608Metric, F.Cu at (83.9, 108.1)
- added R21: 100E, Resistor_SMD:R_0603_1608Metric, F.Cu at (83.9, 110.6)
- added R22: 100E, Resistor_SMD:R_0603_1608Metric, F.Cu at (83.9, 113.1)
- added R23: 100E, Resistor_SMD:R_0603_1608Metric, F.Cu at (87.9, 100.5)
- added R24: 100E, Resistor_SMD:R_0603_1608Metric, F.Cu at (87.9, 103.0)
- added R25: 100E, Resistor_SMD:R_0603_1608Metric, F.Cu at (87.9, 105.5)
- added R26: 1k, Resistor_SMD:R_0603_1608Metric, F.Cu at (93.4, 123.3)
- added R27: 75E, Resistor_SMD:R_0603_1608Metric, B.Cu at (128.9, 101.9)
- added R28: 75E, Resistor_SMD:R_0603_1608Metric, B.Cu at (144.0, 102.0)
- added R29: 75E, Resistor_SMD:R_0603_1608Metric, B.Cu at (138.1, 101.9)
- added R3: 200E, Resistor_SMD:R_0603_1608Metric, F.Cu at (167.7, 93.0)
- added R30: 75E, Resistor_SMD:R_0603_1608Metric, B.Cu at (145.7, 102.0)
- added R31: 75E, Resistor_SMD:R_0603_1608Metric, B.Cu at (133.2, 101.9)
- added R32: 75E, Resistor_SMD:R_0603_1608Metric, B.Cu at (131.4, 102.0)
- added R33: 75E, Resistor_SMD:R_0603_1608Metric, B.Cu at (150.6, 102.0)
- added R34: 75E, Resistor_SMD:R_0603_1608Metric, B.Cu at (148.1, 102.0)
- added R35: 1k, Resistor_SMD:R_0603_1608Metric, F.Cu at (93.4, 125.8)
- added R36: 10k, Resistor_SMD:R_0603_1608Metric, F.Cu at (93.4, 128.3)
- added R4: 200E, Resistor_SMD:R_0603_1608Metric, F.Cu at (169.5, 91.7)
- added R5: 200E, Resistor_SMD:R_0603_1608Metric, F.Cu at (171.8, 90.2)
- added R6: 200E, Resistor_SMD:R_0603_1608Metric, F.Cu at (179.4, 93.6)
- added R7: 100E, Resistor_SMD:R_0603_1608Metric, F.Cu at (166.1, 93.0)
- added R8: 100E, Resistor_SMD:R_0603_1608Metric, F.Cu at (170.1, 104.1)
- added R9: 100E, Resistor_SMD:R_0603_1608Metric, F.Cu at (173.8, 104.1)
- added S1: EVQ-P7A01P, Library:SW_EVQ-P7A01P, B.Cu at (160.4, 71.3)
- added S2: PTS526SM20SMTR21_LFS, Library:PTS526SM20SMTR21LFS, F.Cu at (159.6, 74.2)
- added VR1: AP7366EA-33W5-7, Library:SOT-25-AP7366EA, F.Cu at (111.3, 94.0)
- added X2: SS-53000-001, Library:STEWART_SS-53000-001, F.Cu at (172.7, 77.2)
- C103, C203: value 1uF 10V -> 4.7uF; footprint Capacitor_Tantalum_SMD:CP_EIA-3216-10_Kemet-I_Pad1.58x1.35mm_HandSolder -> Capacitor_SMD:C_0603_1608Metric
- C105, C23, C29: value 10uF 10V -> 4.7uF; footprint Capacitor_Tantalum_SMD:CP_EIA-3216-10_Kemet-I_Pad1.58x1.35mm_HandSolder -> Capacitor_SMD:C_0603_1608Metric
- C15, C18, C30: value 100nF -> 4.7uF
- C2, C3: value 10uF 10V -> 100nF; footprint Capacitor_Tantalum_SMD:CP_EIA-3216-10_Kemet-I_Pad1.58x1.35mm_HandSolder -> Capacitor_SMD:C_0603_1608Metric; moved to F.Cu
- C22: value 10uF 10V -> 4.7uF; footprint Capacitor_Tantalum_SMD:CP_EIA-3216-10_Kemet-I_Pad1.58x1.35mm_HandSolder -> Capacitor_SMD:C_0603_1608Metric; moved to F.Cu
- C36: value 2.2nF -> 4.7uF; moved to F.Cu
- C6, C8: moved to F.Cu
- R55: moved to B.Cu
- U1: value 10CL025YE144C8G -> SOM_FPGA_LP; footprint Library:QFP50P2200X2200X165-145N -> Library:SOM_FPGA_LP
- U4: value M25P80-VMN3TPB -> MAX3814; footprint Package_SO:SO-8_3.9x4.9mm_P1.27mm -> Package_QFP:TQFP-32_5x5mm_P0.5mm
- U6: value AT93C46DN-SH-T -> ESP32-S3-WROOM-1-N8R8; footprint Package_SO:SO-8_3.9x4.9mm_P1.27mm -> Library:MODULE_ESP32-S3-WROOM-1-N8R8; moved to B.Cu
- X3: value 302-S101 -> 490107671012_JTAG; footprint Library:302-S101 -> Library:490107671012
- moved C18 94.1 mm to (96.7, 105.0), turned to 90 degrees
- moved R72 93.2 mm to (170.9, 121.4)
- moved C2 66.1 mm to (166.8, 95.3), turned to 0 degrees
- moved C44 64.7 mm to (132.9, 113.5)
- moved C21 64.0 mm to (129.4, 108.9)
- moved C30 49.0 mm to (135.3, 108.5)
- moved C10 48.0 mm to (179.7, 95.4), turned to 180 degrees
- moved C15 46.4 mm to (129.4, 106.4)
- moved C3 45.8 mm to (166.9, 96.9), turned to 0 degrees
- moved C37 44.6 mm to (93.4, 118.2)
- moved C38 44.6 mm to (93.4, 120.7)
- moved R55 44.5 mm to (121.5, 93.3), turned to -90 degrees
- moved U6 35.2 mm to (180.6, 102.9), turned to 90 degrees
- moved U4 33.2 mm to (173.1, 95.5), turned to 90 degrees
- moved C14 26.8 mm to (171.1, 113.9)
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Connections:
- AX2 pad 2: Net-(C203-MINUS) -> Net-(AX2-Pad2)
- AX2 pad 3: Net-(C203-MINUS) -> Net-(AX2-Pad2)
- AX2 pad 4: Net-(C103-MINUS) -> Net-(AX2-Pad4)
- AX2 pad 5: Net-(C103-MINUS) -> Net-(AX2-Pad4)
- C10 pad 1: +3.3V -> /LVDS_CLK_N
- C10 pad 2: GND -> Net-(U4-IND-)
- C103 pad 1: Net-(C103-PLUS) -> Net-(AX2-Pad4)
- C103 pad 2: Net-(C103-MINUS) -> Net-(C103-Pad2)
- C105 pad 1: +3.3VDAC -> GNDA
- C105 pad 2: GNDA -> +3.3VDAC
- C11 pad 1: +1V2 -> +3.3V
- C12 pad 1: Net-(U1-VCCA1) -> GND
- C12 pad 2: GND -> +3.3V
- C13 pad 1: +2V5 -> GND
- C13 pad 2: GND -> +3.3V
- C14 pad 1: +2V5 -> GND
- C14 pad 2: GND -> +3.3V
- C15 pad 1: Net-(U1-VCCA3) -> GND
- C15 pad 2: GND -> +3V3
- C18 pad 1: +1V2 -> /SLTSOUND
- C18 pad 2: GND -> Net-(C18-Pad2)
- C19 pad 2: +1V2 -> +3.3V
- C2 pad 1: GND -> /LVDS_D2_P
- C2 pad 2: +3V3 -> Net-(U4-INA+)
- C20 pad 1: +1V2 -> +5V
- C203 pad 1: Net-(C203-PLUS) -> Net-(AX2-Pad2)
- C203 pad 2: Net-(C203-MINUS) -> Net-(C203-Pad2)
- C21 pad 1: +2V5 -> GND
- C21 pad 2: GND -> +3V3
- C3 pad 1: GND -> /LVDS_D2_N
- C3 pad 2: +1V2 -> Net-(U4-INA-)
- C30 pad 2: +3.3V -> +5V
- C36 pad 1: Net-(C36-Pad1) -> GND
- C36 pad 2: GNDA -> +3.3V
- C37 pad 1: Net-(U1-VCCA2) -> GND
- C37 pad 2: GND -> +3.3V
- C38 pad 1: Net-(U1-VCCA4) -> GND
- C38 pad 2: GND -> /PUSH_BUTTON
- C44 pad 1: Net-(U1-VCCD_PLL2) -> +5V
- C6 pad 1: GND -> /LVDS_D0_P
- C6 pad 2: +1V2 -> Net-(U4-INC+)
- C7 pad 1: +3.3V -> +5V
- C8 pad 1: +3.3V -> /LVDS_D0_N
- C8 pad 2: GND -> Net-(U4-INC-)
- C9 pad 1: GND -> /LVDS_CLK_P
- C9 pad 2: +3V3 -> Net-(U4-IND+)
- R103 pad 2: Net-(C103-PLUS) -> Net-(C103-Pad2)
- R203 pad 2: Net-(C203-PLUS) -> Net-(C203-Pad2)
- U1 pad 1: Net-(U1-VCCD_PLL3) -> +5V
- U1 pad 10: /DAC_DIN -> /TDI
- U1 pad 102: +1V2 -> unconnected-(U1-B5-IO8N-Pad102)
- U1 pad 104: GND -> unconnected-(U1-B5-IO9P-Pad104)
- U1 pad 107: Net-(U1-VCCA2) -> unconnected-(U1-B6-IO9-Pad107)
- U1 pad 108: GND -> unconnected-(U1-B6-IO1P-Pad108)
- U1 pad 109: Net-(U1-VCCD_PLL2) -> +IO2V5
- U1 pad 11: /DAC_BCK -> unconnected-(U1-+3V3-Pad11)
- U1 pad 110: GND -> /PUSH_BUTTON
- U1 pad 111: unconnected-(U1-IO_44-Pad111) -> +IO2V5
- U1 pad 112: unconnected-(U1-IO_45-Pad112) -> /HDDLED
- U1 pad 113: unconnected-(U1-IO_46-Pad113) -> +IO1V8
- U1 pad 114: unconnected-(U1-IO_47-Pad114) -> +IO2V5
- U1 pad 115: unconnected-(U1-IO_48-Pad115) -> +IO1V8
- U1 pad 116: +1V2 -> +IO3V3
- U1 pad 117: +3.3V -> +IO3V3
- U1 pad 118: GND -> +IO3V3
- U1 pad 119: unconnected-(U1-IO_49-Pad119) -> +IO3V3
- U1 pad 12: /DCLK -> /TCK
- U1 pad 120: unconnected-(U1-IO_50-Pad120) -> +IO3V3
- U1 pad 121: unconnected-(U1-IO_51-Pad121) -> GND
- U1 pad 122: +3.3V -> GND
- U1 pad 124: +1V2 -> GND
- U1 pad 13: /DATA0 -> unconnected-(U1-+3V3-Pad13)
- U1 pad 14: /nCONFIG -> /TMS
- U1 pad 15: /TDI -> unconnected-(U1-+3V3-Pad15)
- U1 pad 16: /TCK -> /TDO
- U1 pad 17: +3.3V -> unconnected-(U1-B1-CLK1-Pad17)
- U1 pad 18: /TMS -> /JTAGVCC
- U1 pad 19: GND -> /~{SLT_BUSDIR}
- U1 pad 20: /TDO -> /LVDS_D2_N
- U1 pad 21: /nCE -> /~{SLT_INT}
- U1 pad 22: /ADC_DOUT -> /LVDS_D2_P
- U1 pad 23: GND -> /~{SLT_WAIT}
- U1 pad 24: GND -> /LVDS_D1_N
- U1 pad 25: /CLC50 -> /SLT_CLC
- U1 pad 26: +3.3V -> /LVDS_D1_P
- U1 pad 27: GND -> /~{SLT_SLTSL}
- U1 pad 28: /DAC_SCK -> /LVDS_D0_N
- U1 pad 29: +1V2 -> /~{SLT_RFSH}
- U1 pad 3: Net-(U1-VCCA3) -> +5V
- U1 pad 30: unconnected-(U1-GND_4-Pad30) -> /LVDS_D0_P
- U1 pad 31: /DAC_BCK -> /SLT_MUX
- U1 pad 32: /DAC_SCK -> /LVDS_CLK_N
- U1 pad 33: /DAC_FLT -> /SLT_X7
- U1 pad 34: +1V2 -> /LVDS_CLK_P
- U1 pad 35: Net-(U1-VCCA1) -> /SLT_X6
- U1 pad 36: GND -> unconnected-(U1-B2-IO9N-Pad36)
- U1 pad 37: Net-(U1-VCCD_PLL1) -> /SLT_X5
- U1 pad 38: +1V2 -> /~{SLT_RESET}
- U1 pad 39: /SLT_X7 -> /SLT_X4
- U1 pad 40: +3.3V -> /HDMI_SDA
- U1 pad 41: GND -> /SLT_X3
- U1 pad 42: /SLT_X6 -> /HDMI_SCL
- U1 pad 43: /SLT_X5 -> /SLT_X2
- U1 pad 44: /SLT_X4 -> /ADC_BCK
- U1 pad 45: +1V2 -> /SLT_X1
- U1 pad 46: /SLT_X3 -> /ADC_LRCK
- U1 pad 47: +3.3V -> /SLT_X0
- U1 pad 48: GND -> /ADC_SCKI
- U1 pad 49: /SLT_X2 -> /SLT_Y7
- U1 pad 5: +1V2 -> +5V
- U1 pad 50: /SLT_X1 -> /ADC_DOUT
- U1 pad 51: /SLT_X0 -> /SLT_Y6
- U1 pad 52: /SLT_Y7 -> /DAC_SCK
- U1 pad 53: /SLT_Y6 -> /SLT_Y5
- U1 pad 54: /SLT_Y5 -> /DAC_BCK
- U1 pad 56: +3.3V -> /DAC_SCK
- U1 pad 57: GND -> /SLT_Y3
- U1 pad 58: /SLT_MUX -> /DAC_FLT
- U1 pad 59: /SLT_Y0 -> /SLT_Y2
- U1 pad 6: /ASDO -> GND
- U1 pad 60: /SLT_Y2 -> /DAC_XSMT
- U1 pad 61: +1V2 -> /SLT_Y1
- U1 pad 62: +3.3V -> /DAC_LRCK
- U1 pad 63: GND -> /SLT_Y0
- U1 pad 64: GND -> /DAC_DIN
- U1 pad 65: /SLT_Y1 -> unconnected-(U1-B4-CLK12-Pad65)
- U1 pad 66: /SLT_Y3 -> /DAC_BCK
- U1 pad 67: /~{SLT_RFSH} -> unconnected-(U1-B4-IO9-Pad67)
- U1 pad 68: /~{SLT_WAIT} -> /SD_CLK
- U1 pad 69: /~{SLT_RESET} -> unconnected-(U1-B4-IO6-Pad69)
- U1 pad 7: /DAC_LRCK -> +5V
- U1 pad 70: +1V2 -> /SD_CMD
- U1 pad 71: /~{SLT_BUSDIR} -> unconnected-(U1-B4-IO11-Pad71)
- U1 pad 72: /~{SLT_INT} -> /SD_DAT0
- U1 pad 73: Net-(U1-VCCD_PLL4) -> /SND5
- U1 pad 74: GND -> /SD_DAT1
- U1 pad 75: Net-(U1-VCCA4) -> /SND4
- U1 pad 76: /~{SLT_SLTSL} -> /SD_DAT2
- U1 pad 77: unconnected-(U1-IO_31-Pad77) -> /SND3
- U1 pad 78: +1V2 -> /SD_DAT3
- U1 pad 79: unconnected-(U1-GND_10-Pad79) -> /SND2
- U1 pad 8: /nCS0 -> GND
- U1 pad 80: unconnected-(U1-IO_32-Pad80) -> /SD_WP
- U1 pad 81: +3.3V -> /SND1
- U1 pad 82: GND -> /SD_CD
- U1 pad 83: unconnected-(U1-IO_33-Pad83) -> /SND0
- U1 pad 84: +1V2 -> unconnected-(U1-B4-IO12-COP-Pad84)
- U1 pad 88: /SLT_CLC -> unconnected-(U1-B5-IO4P-Pad88)
- U1 pad 89: GND -> unconnected-(U1-B6-IO2-Pad89)
- U1 pad 9: /nSTATUS -> +3.3V
- U1 pad 90: GND -> unconnected-(U1-B5-IO4N-Pad90)
- U1 pad 91: GND -> unconnected-(U1-B6-IO6-Pad91)
- U1 pad 92: /CONF_DONE -> unconnected-(U1-B5-IO3P-Pad92)
- U1 pad 93: +3.3V -> unconnected-(U1-B6-IO3-Pad93)
- U1 pad 94: GND -> unconnected-(U1-B5-IO3N-Pad94)
- U1 pad 95: GND -> unconnected-(U1-B6-IO4-Pad95)
- U1 pad 96: +2V5 -> unconnected-(U1-B5-IO7P-Pad96)
- U1 pad 97: GND -> unconnected-(U1-B6-CLK5-Pad97)
- U14 pad 10: +3V3 -> +2V5
- U14 pad 2: +3V3 -> +2V5
- U2 pad 1: /~{SLT_MUX} -> /SLT_MUX
- U2 pad 19: /~{SLT_MUX} -> /SLT_MUX
- U4 pad 1: /nCSO -> unconnected-(U4-NC-Pad1)
- U4 pad 3: +3.3V -> Net-(U4-INB-)
- U4 pad 4: GND -> +3.3V
- U4 pad 5: /ASDO -> +3.3V
- U4 pad 6: /DCLK -> Net-(U4-INC+)
- U4 pad 7: +3.3V -> Net-(U4-INC-)
- U4 pad 8: +3.3V -> unconnected-(U4-NC-Pad8)
- U6 pad 1: /EECS -> GND
- U6 pad 2: /EECK -> +3.3V
- U6 pad 3: /EEDI -> /ESP_EN
- U6 pad 4: /EEDO -> /ESP_IO4
- U6 pad 5: GND -> /ESP_IO5
- U6 pad 6: GND -> /ESP_IO6
- U6 pad 7: unconnected-(U6-NC-Pad7) -> /ESP_IO7
- U6 pad 8: +3V3 -> /ESP_IO15
- U8 pad 1: /SLT_MUX -> /~{SLT_MUX}
- U8 pad 19: /SLT_MUX -> /~{SLT_MUX}
- X3 pad 4: +3.3V -> /JTAGVCC
- X3 pad 6: +3.3V -> unconnected-(X3-NC-Pad6)
Routing:
- net /JTAGVCC: track 0.00 -> 59.8 mm, vias 0 -> 1
- net GND: track 279.1 -> 236.0 mm, vias 8 -> 9
- net +3V3: track 179.2 -> 139.5 mm, vias 12 -> 10
- net +5V: track 159.7 -> 134.5 mm, vias 10 -> 9
- net /SLT_MUX: track 63.3 -> 38.9 mm, vias 5 -> 3
- net /ADC_DOUT: track 23.9 -> 3.37 mm, vias 2 -> 0
- net +1V2: track 20.0 -> 0.00 mm, vias 1 -> 0
- net /SLT_Y5: track 18.5 -> 0.00 mm, vias 1 -> 0
- net /SLT_Y4: track 18.4 -> 0.00 mm, vias 1 -> 0
- net /~{SLT_RFSH}: track 18.2 -> 0.00 mm
- net /SLT_CLC: track 18.1 -> 0.00 mm
- net Net-(AX2-Pad2): track 0.00 -> 18.0 mm
- net Net-(C203-MINUS): track 18.0 -> 0.00 mm
- net /~{SLT_WAIT}: track 16.5 -> 0.06 mm
- net +3.3VDAC: track 45.0 -> 29.2 mm
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Other:
- board text removed: "-"
- board text removed: "CY62167DV30"
- board text removed: "EPCS4SI8 or M25P80"
- board text removed: "M29W640"
- board text removed: "SG-310 50 MHz"

Commit message: Schematic work in progress
Parts:
- removed AX3: SJ1-3523N, Library:ST-222_1
- removed C101, C201: 2.2nF, Capacitor_SMD:C_0603_1608Metric
- removed C102: 100nF, Capacitor_SMD:C_0603_1608Metric
- removed C104, C204: 2.2uF, Capacitor_SMD:C_0603_1608Metric
- removed C203: 4.7uF, Capacitor_SMD:C_0603_1608Metric
- removed C205: 10uF 10V, Capacitor_Tantalum_SMD:CP_EIA-3216-10_Kemet-I_Pad1.58x1.35mm_HandSolder
- removed R103, R203: 75E, Resistor_SMD:R_0603_1608Metric
- removed R104, R204: 470E, Resistor_SMD:R_0603_1608Metric
- removed R55: 220E, Resistor_SMD:R_0603_1608Metric
- removed R64: 10E, Resistor_SMD:R_0603_1608Metric
- removed S2: PTS526SM20SMTR21_LFS, Library:PTS526SM20SMTR21LFS
- added C39: 4.7uF, Capacitor_SMD:C_0603_1608Metric, F.Cu at (107.8, 98.1)
- added C40: 4.7uF, Capacitor_SMD:C_0603_1608Metric, F.Cu at (107.8, 100.6)
- added C41: 1uF, Capacitor_SMD:C_0603_1608Metric, F.Cu at (207.1, 99.2)
- added C42: 100nF, Capacitor_SMD:C_0603_1608Metric, F.Cu at (207.1, 101.8)
- added C43: 100nF, Capacitor_SMD:C_0603_1608Metric, F.Cu at (160.2, 114.0)
- added C46: 100nF, Capacitor_SMD:C_0603_1608Metric, F.Cu at (211.1, 94.2)
- added C47: 100nF, Capacitor_SMD:C_0603_1608Metric, F.Cu at (211.1, 96.7)
- added C48: 1uF, Capacitor_SMD:C_0603_1608Metric, F.Cu at (211.1, 99.2)
- added C49: 1uF, Capacitor_SMD:C_0603_1608Metric, F.Cu at (211.1, 101.8)
- added C50: 1uF, Capacitor_SMD:C_0603_1608Metric, F.Cu at (215.1, 91.7)
- added C51: 1uF, Capacitor_SMD:C_0603_1608Metric, F.Cu at (215.1, 94.2)
- added J3: UJ20-C-H-G-SMT-2-P16-TR, Library:SAMESKY_UJ20-C-H-G-SMT-2-P16-TR, F.Cu at (157.8, 69.8)
- added J4: UJ20-C-H-G-SMT-2-P16-TR, Library:SAMESKY_UJ20-C-H-G-SMT-2-P16-TR, F.Cu at (188.3, 69.8)
- added J5: Conn_01x08, Connector_PinHeader_2.00mm:PinHeader_1x08_P2.00mm_Vertical, F.Cu at (96.8, 88.5)
- added J6: Conn_01x06, Connector_PinHeader_2.00mm:PinHeader_1x06_P2.00mm_Vertical, F.Cu at (120.7, 91.2)
- added J7: Conn_02x04_Odd_Even, Connector_PinHeader_2.00mm:PinHeader_2x04_P2.00mm_Vertical, F.Cu at (186.1, 91.7)
- added Q1: UM6K34NTCN, Package_TO_SOT_SMD:SOT-363_SC-70-6, F.Cu at (176.2, 84.7)
- added R12: 10k, Resistor_SMD:R_0603_1608Metric, B.Cu at (171.7, 84.5)
- added R37: 10k, Resistor_SMD:R_0603_1608Metric, B.Cu at (167.8, 82.0)
- added R38: 10k, Resistor_SMD:R_0603_1608Metric, F.Cu at (179.3, 87.8)
- added R39: 10k, Resistor_SMD:R_0603_1608Metric, F.Cu at (215.1, 101.8)
- added R43: 1k, Resistor_SMD:R_0603_1608Metric, B.Cu at (175.4, 87.6)
- added R44: 1k, Resistor_SMD:R_0603_1608Metric, B.Cu at (166.4, 81.5)
- added R46: 5k1, Resistor_SMD:R_0603_1608Metric, F.Cu at (184.3, 85.6)
- added R47: 5k1, Resistor_SMD:R_0603_1608Metric, B.Cu at (186.7, 73.7)
- added R48: 5k1, Resistor_SMD:R_0603_1608Metric, B.Cu at (156.0, 73.2)
- added R49: 5k1, Resistor_SMD:R_0603_1608Metric, B.Cu at (159.4, 73.3)
- added R50: 10k, Resistor_SMD:R_0603_1608Metric, F.Cu at (148.1, 79.8)
- added S3: EVQ-P7A01P, Library:SW_EVQ-P7A01P, F.Cu at (135.9, 71.2)
- added U7: MCP2221AT-I/SL, Package_SO:SOIC-14_3.9x8.7mm_P1.27mm, F.Cu at (170.2, 84.5)
- C1, C28: value 10uF 10V -> 4.7uF; footprint Capacitor_Tantalum_SMD:CP_EIA-3216-10_Kemet-I_Pad1.58x1.35mm_HandSolder -> Capacitor_SMD:C_0603_1608Metric
- C103: value 4.7uF -> 1uF
- C11, C15, C19, C20, C21, C24, C44, R14, R15, R16, R17, R18, R19, R20, R21, R22, R23, R24, R25: moved to B.Cu
- C25: value 100nF -> 4.7uF
- C26: value 10uF 10V -> 100nF; footprint Capacitor_Tantalum_SMD:CP_EIA-3216-10_Kemet-I_Pad1.58x1.35mm_HandSolder -> Capacitor_SMD:C_0603_1608Metric
- C27: value 100nF -> 1uF; moved to F.Cu
- C29, C32, S1: moved to F.Cu
- C30: value 4.7uF -> 1uF; moved to F.Cu
- C33, C34, C35: value 100nF -> 1uF
- R26, R35: value 1k -> 10k
- U5: value PCM5101APWR -> NAU88C22A; footprint Package_SO:TSSOP-20_4.4x6.5mm_P0.65mm -> Library:QFN-32-NAU88C22YG
- U9: value PCM1808PWR -> AP22816AKEWT; footprint Package_SO:TSSOP-14_4.4x5mm_P0.65mm -> Package_TO_SOT_SMD:SOT-23-5
- moved R26 124.6 mm to (215.1, 96.7)
- moved R35 124.6 mm to (215.1, 99.2)
- moved C37 92.2 mm to (185.0, 108.2), turned to 180 degrees
- moved C36 91.8 mm to (185.0, 109.8), turned to 180 degrees
- moved C27 90.1 mm to (203.0, 94.2)
- moved C35 86.8 mm to (207.1, 96.7), turned to 0 degrees
- moved C34 86.5 mm to (207.1, 94.2), turned to 0 degrees
- moved R36 84.0 mm to (162.1, 79.8)
- moved C32 81.1 mm to (203.0, 101.8)
- moved C31 81.1 mm to (203.0, 99.2), turned to 0 degrees
- moved R19 77.1 mm to (161.0, 104.9), turned to -90 degrees
- moved C38 76.9 mm to (158.4, 79.8)
- moved R16 76.8 mm to (156.3, 104.9), turned to -90 degrees
- moved R18 75.5 mm to (159.4, 104.9), turned to -90 degrees
- moved R15 75.0 mm to (154.7, 104.9), turned to -90 degrees
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Connections:
- C1 pad 1: GND -> +5V
- C10 pad 1: /LVDS_CLK_N -> Net-(U4-IND-)
- C10 pad 2: Net-(U4-IND-) -> /LVDS_CLK_N
- C103 pad 1: Net-(AX2-Pad4) -> Net-(U5-LAUXIN)
- C103 pad 2: Net-(C103-Pad2) -> Net-(AX2-Pad4)
- C105 pad 1: GNDA -> +5V
- C105 pad 2: +3.3VDAC -> +3V3DAC
- C11 pad 1: +3.3V -> +5V
- C11 pad 2: GND -> +3.3V
- C12 pad 1: GND -> +3.3V
- C12 pad 2: +3.3V -> +5V
- C13 pad 1: GND -> +3.3V
- C13 pad 2: +3.3V -> +5V
- C14 pad 1: GND -> +3.3V
- C14 pad 2: +3.3V -> +5V
- C15 pad 1: GND -> +5V
- C16 pad 1: +3V3 -> +5V
- C16 pad 2: GND -> +3V3
- C17 pad 1: +3V3 -> +5V
- C17 pad 2: GND -> +3V3
- C19 pad 1: GND -> +3.3V
- C19 pad 2: +3.3V -> +5V
- C2 pad 1: /LVDS_D2_P -> Net-(U4-INA+)
- C2 pad 2: Net-(U4-INA+) -> /LVDS_D2_P
- C20 pad 2: GND -> +5V
- C21 pad 1: GND -> +5V
- C22 pad 1: GND -> +5V
- C22 pad 2: +3.3VDAC -> +3V3DAC
- C23 pad 1: GND -> GNDA
- C24 pad 1: GNDA -> +5V
- C24 pad 2: +3.3VDAC -> +3V3
- C25 pad 1: GND -> +5V
- C25 pad 2: +3V3 -> /USB_VBUS
- C26 pad 1: GNDA -> +5V
- C26 pad 2: +3.3VDAC -> /USB_VBUS
- C27 pad 1: GNDA -> +5V
- C27 pad 2: +3.3VDAC -> +5V
- C28 pad 1: GNDA -> Net-(U5-VREF)
- C28 pad 2: Net-(C28-PLUS) -> GNDA
- C29 pad 1: GNDA -> Net-(U5-MICBIAS)
- C29 pad 2: Net-(U9-VCC) -> GNDA
- C3 pad 1: /LVDS_D2_N -> Net-(U4-INA-)
- C3 pad 2: Net-(U4-INA-) -> /LVDS_D2_N
- C30 pad 1: GND -> +5V
- C31 pad 1: GNDA -> /ESP_BOOT_MODE
- C31 pad 2: Net-(C28-PLUS) -> +5V
- C32 pad 1: GNDA -> +5V
- C32 pad 2: Net-(U9-VinR) -> +5V
- C33 pad 1: GNDA -> Net-(U5-RAUXIN)
- C33 pad 2: Net-(U9-VinL) -> Net-(AX2-Pad2)
- C34 pad 1: GND -> Net-(AX1-Pad4)
- C34 pad 2: +3V3 -> Net-(U5-AUXOUT1)
- C35 pad 1: GNDA -> Net-(AX1-Pad2)
- C35 pad 2: Net-(U9-VCC) -> Net-(U5-AUXOUT2)
- C36 pad 1: GND -> +5V
- C37 pad 1: GND -> +3.3V
- C37 pad 2: +3.3V -> +5V
- C38 pad 1: GND -> /PUSH_BUTTON
- C38 pad 2: /PUSH_BUTTON -> +5V
- C4 pad 1: /LVDS_D1_P -> Net-(U4-INB+)
- C4 pad 2: Net-(U4-INB+) -> /LVDS_D1_P
- C44 pad 2: GND -> +5V
- C45 pad 1: +3V3 -> +5V
- C45 pad 2: GND -> +3V3
- C5 pad 1: /LVDS_D1_N -> Net-(U4-INB-)
- C5 pad 2: Net-(U4-INB-) -> /LVDS_D1_N
- C6 pad 1: /LVDS_D0_P -> Net-(U4-INC+)
- C6 pad 2: Net-(U4-INC+) -> /LVDS_D0_P
- C7 pad 2: GND -> +5V
- C8 pad 1: /LVDS_D0_N -> Net-(U4-INC-)
- C8 pad 2: Net-(U4-INC-) -> /LVDS_D0_N
- C9 pad 1: /LVDS_CLK_P -> Net-(U4-IND+)
- C9 pad 2: Net-(U4-IND+) -> /LVDS_CLK_P
- J1 pad 1: GND -> +5V
- J2 pad 3: GND -> +5V
- J2 pad 6: GND -> +5V
- J2 pad G1: GND -> +5V
- J2 pad G2: GND -> +5V
- LED1 pad 1: /HDDLED -> Net-(LED1-K)
- LED1 pad 2: Net-(LED1-A) -> +3.3V
- MP1 pad 1: GND -> +5V
- R11 pad 1: GND -> +5V
- R13 pad 1: GND -> +5V
- R26 pad 1: /DBG_TXD -> +3.3V
- R26 pad 2: Net-(AX3-Pad4) -> /ESP_BOOT_MODE
- R35 pad 1: /DBG_RXD -> Net-(AX1-Pad4)
- R35 pad 2: Net-(AX3-Pad2) -> GNDA
- R45 pad 1: +3.3V -> Net-(LED1-K)
- R45 pad 2: Net-(LED1-A) -> /HDDLED
- R72 pad 2: GND -> +5V
- R99 pad 1: GND -> +5V
- S1 pad 2: GND -> +5V
- U1 pad 100: unconnected-(U1-B5-IO8P-Pad100) -> /ESP_IO39
- U1 pad 101: unconnected-(U1-B6-IO8-Pad101) -> /ESP_IO7
- U1 pad 102: unconnected-(U1-B5-IO8N-Pad102) -> /ESP_IO11
- U1 pad 103: unconnected-(U1-B6-IO7-Pad103) -> /ESP_IO8
- U1 pad 104: unconnected-(U1-B5-IO9P-Pad104) -> /ESP_IO12
- U1 pad 105: unconnected-(U1-B6-IO5-Pad105) -> /ESP_IO9
- U1 pad 106: unconnected-(U1-B5-IO9N-Pad106) -> /ESP_IO13
- U1 pad 107: unconnected-(U1-B6-IO9-Pad107) -> /ESP_IO10
- U1 pad 108: unconnected-(U1-B6-IO1P-Pad108) -> /ESP_IO14
- U1 pad 11: unconnected-(U1-+3V3-Pad11) -> +3.3V
- U1 pad 110: /PUSH_BUTTON -> /ESP_IO15
- U1 pad 112: /HDDLED -> /ESP_IO16
- U1 pad 121: GND -> +5V
- U1 pad 122: GND -> +5V
- U1 pad 123: GND -> +5V
- U1 pad 124: GND -> +5V
- U1 pad 13: unconnected-(U1-+3V3-Pad13) -> +3.3V
- U1 pad 15: unconnected-(U1-+3V3-Pad15) -> +3.3V
- U1 pad 2: GND -> +5V
- U1 pad 36: unconnected-(U1-B2-IO9N-Pad36) -> /HDDLED
- U1 pad 4: GND -> +5V
- U1 pad 44: /ADC_BCK -> /CODEC_MCK
- U1 pad 46: /ADC_LRCK -> /CODEC_BCK
- U1 pad 48: /ADC_SCKI -> /CODEC_FS
- U1 pad 50: /ADC_DOUT -> /CODEC_DACIN
- U1 pad 52: /DAC_SCK -> /CODEC_ADCOUT
- U1 pad 54: /DAC_BCK -> /CODEC_SCLK
- U1 pad 56: /DAC_SCK -> /CODEC_SDIO
- U1 pad 58: /DAC_FLT -> /CODEC_CSB
- U1 pad 6: GND -> +5V
- U1 pad 60: /DAC_XSMT -> /CODEC_MODE
- U1 pad 62: /DAC_LRCK -> /ESP_IO21/USBEN
- U1 pad 64: /DAC_DIN -> /SD_CLK
- U1 pad 65: unconnected-(U1-B4-CLK12-Pad65) -> /DBG_RXD
- U1 pad 66: /DAC_BCK -> /SD_CMD
- U1 pad 67: unconnected-(U1-B4-IO9-Pad67) -> /DBG_TXD
- U1 pad 68: /SD_CLK -> /SD_DAT0
- U1 pad 69: unconnected-(U1-B4-IO6-Pad69) -> /~{DBG_ACT}
- U1 pad 70: /SD_CMD -> /SD_DAT1
- U1 pad 71: unconnected-(U1-B4-IO11-Pad71) -> /PUSH_BUTTON
- U1 pad 72: /SD_DAT0 -> /SD_DAT2
- U1 pad 74: /SD_DAT1 -> /SD_DAT3
- U1 pad 76: /SD_DAT2 -> /SD_WP
- U1 pad 78: /SD_DAT3 -> /SD_CD
- U1 pad 8: GND -> +5V
- U1 pad 80: /SD_WP -> /DBG_SCL
- U1 pad 82: /SD_CD -> /DBG_SDA
- U1 pad 84: unconnected-(U1-B4-IO12-COP-Pad84) -> /ESP_TXD
- U1 pad 85: unconnected-(U1-B5-IO11-Pad85) -> /ESP_EN
- U1 pad 86: unconnected-(U1-B4-IO12-CON-Pad86) -> /ESP_RXD
- U1 pad 87: unconnected-(U1-B5-IO10-Pad87) -> /ESP_BOOT_MODE
- U1 pad 88: unconnected-(U1-B5-IO4P-Pad88) -> /ESP_IO17/SCL
- U1 pad 89: unconnected-(U1-B6-IO2-Pad89) -> /ESP_IO1
- U1 pad 90: unconnected-(U1-B5-IO4N-Pad90) -> /ESP_IO18/SDA
- U1 pad 91: unconnected-(U1-B6-IO6-Pad91) -> /ESP_IO2
- U1 pad 92: unconnected-(U1-B5-IO3P-Pad92) -> /ESP_IO35/GP0
- U1 pad 93: unconnected-(U1-B6-IO3-Pad93) -> /ESP_IO3
- U1 pad 94: unconnected-(U1-B5-IO3N-Pad94) -> /ESP_IO36/GP1
- U1 pad 95: unconnected-(U1-B6-IO4-Pad95) -> /ESP_IO4
- U1 pad 96: unconnected-(U1-B5-IO7P-Pad96) -> /ESP_IO37/GP2
- U1 pad 97: unconnected-(U1-B6-CLK5-Pad97) -> /ESP_IO5
- U1 pad 98: unconnected-(U1-B5-IO7N-Pad98) -> /ESP_IO38/GP3
- U1 pad 99: unconnected-(U1-B6-CLK4-Pad99) -> /ESP_IO6
- U10 pad 3: GND -> +5V
- U12 pad 11: GND -> +5V
- U14 pad 11: GND -> +5V
- U2 pad 10: GND -> +5V
- U3 pad 10: GND -> +5V
- U4 pad 12: GND -> +5V
- U4 pad 13: GND -> +5V
- U4 pad 16: GND -> +5V
- U4 pad 20: GND -> +5V
- U4 pad 21: GND -> +5V
- U4 pad 25: GND -> +5V
- U4 pad 28: GND -> +5V
- U5 pad 1: +3.3VDAC -> Net-(U5-LMICP)
- U5 pad 10: GND -> /CODEC_DACIN
- U5 pad 11: /DAC_FLT -> /CODEC_MCK
- U5 pad 12: /DAC_SCK -> GNDA
- U5 pad 13: /DAC_BCK -> +IO1V8
- U5 pad 14: /DAC_DIN -> +3V3
- U5 pad 15: /DAC_LRCK -> /CODEC_CSB
- U5 pad 16: GND -> /CODEC_SCLK
- U5 pad 17: /DAC_XSMT -> /CODEC_SDIO
- U5 pad 18: Net-(C205-PLUS) -> /CODEC_MODE
- U5 pad 19: GND -> Net-(U5-LAUXIN)
- U5 pad 20: +3V3 -> Net-(U5-RAUXIN)
- U5 pad 3: GNDA -> Net-(J5-Pin_1)
- U5 pad 7: Net-(U5-OUTR) -> /CODEC_FS
- U5 pad 8: +3.3VDAC -> /CODEC_BCK
- U5 pad 9: GNDA -> /CODEC_ADCOUT
- U6 pad 1: GND -> +5V
- U6 pad 10: /ESP_IO17 -> /ESP_IO17/SCL
- U6 pad 11: /ESP_IO18 -> /ESP_IO18/SDA
- U6 pad 13: unconnected-(U6-IO19/USB_Dn-Pad13) -> /ESP_USB_Dn
- U6 pad 14: unconnected-(U6-IO20/USB-Dp-Pad14) -> /ESP_USB_Dp
- U6 pad 23: /ESP_IO21 -> /ESP_IO21/USBEN
- U6 pad 28: /ESP_IO35 -> /ESP_IO35/GP0
- U6 pad 29: /ESP_IO36 -> /ESP_IO36/GP1
- U6 pad 30: /ESP_IO37 -> /ESP_IO37/GP2
- U6 pad 31: /ESP_IO38 -> /ESP_IO38/GP3
- U6 pad 40: GND -> +5V
- U6 pad 41: GND -> +5V
- U8 pad 10: GND -> +5V
- U9 pad 1: Net-(C28-PLUS) -> /USB_VBUS
- U9 pad 2: GNDA -> +5V
- U9 pad 3: Net-(U9-VCC) -> unconnected-(U9-~{FLG}-Pad3)
- U9 pad 4: +3V3 -> /ESP_IO21/USBEN
- U9 pad 5: GND -> +5V
- VR1 pad 2: +3.3VDAC -> +3V3DAC
- VR1 pad 3: GND -> +5V
- VR1 pad 5: +3.3VDAC -> +3V3DAC
- X1 pad 41: GND -> +5V
- X1 pad 43: GND -> +5V
- X2 pad 11: GND -> +5V
- X2 pad 17: GND -> +5V
- X2 pad 2: GND -> +5V
- X2 pad 5: GND -> +5V
- X2 pad 8: GND -> +5V
- X2 pad S1: GND -> +5V
- X2 pad S2: GND -> +5V
- X2 pad S3: GND -> +5V
- X2 pad S4: GND -> +5V
- X3 pad 10: GND -> +5V
- X3 pad 2: GND -> +5V
Routing:
- net GND: track 236.0 -> 0.00 mm, vias 9 -> 0
- net GNDA: track 169.6 -> 50.7 mm, vias 4 -> 0
- net (no net): track 0.00 -> 90.4 mm
- net +5V: track 134.5 -> 65.4 mm, vias 9 -> 10
- net +3V3: track 139.5 -> 72.3 mm, vias 10 -> 6
- net /JTAGVCC: track 59.8 -> 0.00 mm, vias 1 -> 0
- net /TDI: track 55.3 -> 0.00 mm
- net /TMS: track 51.5 -> 0.00 mm, vias 1 -> 0
- net Net-(J5-Pin_2): track 51.2 -> 0.00 mm, vias 2 -> 0
- net /TDO: track 49.9 -> 0.00 mm
- net /TCK: track 45.0 -> 0.00 mm
- net /SLTSOUND: track 41.5 -> 0.00 mm
- net Net-(U5-OUTR): track 39.3 -> 0.00 mm, vias 2 -> 0
- net +3.3VDAC: track 29.2 -> 0.00 mm, vias 3 -> 0
- net Net-(U9-VinL): track 12.1 -> 0.00 mm, vias 1 -> 0
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Other:
- board text removed: "AS"
- board text removed: "R60"
