File: board/HyperFusionXC.kicad_pcb (KiCad board)
At the start: 2 copper layers, 99 x 65.6 mm, 134 parts, among them J1 Conn_01x02_Pin, J2 10067847-001RLF, J3 UJ20-C-H-G-SMT-2-P16-TR, J4 UJ20-C-H-G-SMT-2-P16-TR, J5 Conn_01x08, J6 Conn_01x06, J7 Conn_02x04_Odd_Even, Q1 UM6K34NTCN, U1 SOM_FPGA_LP, U10 SN74LVC1G04DCKR, U12 TXS0108EPWR, U14 TXS0108EPWR, U2 74AHC541, U3 74AHC541, U4 MAX3814, U5 NAU88C22A, U6 ESP32-S3-WROOM-1-N8R8, U7 MCP2221AT-I/SL, U8 74AHC541, U9 AP22816AKEWT, X1 EDGE50/MSX, X2 SS-53000-001, X3 490107671012_JTAG

Commit message: Schematic work in progress
Parts:
- added C52: 1uF, Capacitor_SMD:C_0603_1608Metric, B.Cu at (177.2, 82.0)
- added C53: 100nF, Capacitor_SMD:C_0603_1608Metric, B.Cu at (182.5, 82.0)
- added C54: 4.7uF, Capacitor_SMD:C_0603_1608Metric, B.Cu at (181.7, 79.7)
- added R40: 1k, Resistor_SMD:R_0603_1608Metric, B.Cu at (157.7, 71.8)
- added U11: AP22816BKAWT-7, Package_TO_SOT_SMD:SOT-23-5, B.Cu at (179.8, 82.5)
- added U15: TXB0104D, Package_SO:SOIC-14_3.9x8.7mm_P1.27mm, B.Cu at (161.0, 76.4)
- C23, C33, R12, R37, R43, R44, R47: moved to F.Cu
- C30, C45, R1, R2, U7: moved to B.Cu
- J6: value Conn_01x06 -> Conn_01x05; footprint Connector_PinHeader_2.00mm:PinHeader_1x06_P2.00mm_Vertical -> Connector_PinSocket_2.00mm:PinSocket_1x05_P2.00mm_Vertical
- J7: value Conn_02x04_Odd_Even -> Conn_02x05_Odd_Even; footprint Connector_PinHeader_2.00mm:PinHeader_2x04_P2.00mm_Vertical -> Connector_PinHeader_2.00mm:PinHeader_2x05_P2.00mm_Vertical
- R25: value 100E -> 200E
- U9: value AP22816AKEWT -> AP22816BKAWT-7
- moved C50 113.1 mm to (102.3, 99.7), turned to 180 degrees
- moved C51 112.8 mm to (102.3, 97.7), turned to 180 degrees
- moved C49 109.2 mm to (102.3, 91.7), turned to 180 degrees
- moved C48 108.9 mm to (102.3, 93.7), turned to 180 degrees
- moved R39 103.7 mm to (111.8, 92.4), turned to 90 degrees
- moved R35 101.9 mm to (113.4, 92.4), turned to 90 degrees
- moved C32 98.6 mm to (104.7, 109.7)
- moved C35 95.2 mm to (111.8, 95.4), turned to -90 degrees
- moved C34 93.7 mm to (113.4, 95.4), turned to -90 degrees
- moved R26 82.4 mm to (135.8, 74.1)
- moved C47 81.1 mm to (134.0, 122.0), turned to 180 degrees
- moved C31 71.1 mm to (135.9, 76.0)
- moved C46 69.5 mm to (146.2, 119.1), turned to 90 degrees
- moved C30 68.8 mm to (136.0, 112.3), turned to 180 degrees
- moved R50 64.0 mm to (198.7, 119.0)
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Connections:
- C1 pad 1: +5V -> GND
- C105 pad 1: +5V -> GND
- C11 pad 1: +5V -> GND
- C11 pad 2: +3.3V -> +3V3
- C12 pad 1: +3.3V -> +3V3
- C12 pad 2: +5V -> GND
- C13 pad 1: +3.3V -> +3V3
- C13 pad 2: +5V -> GND
- C14 pad 1: +3.3V -> +3V3
- C14 pad 2: +5V -> GND
- C15 pad 1: +5V -> GND
- C16 pad 1: +5V -> GND
- C17 pad 1: +5V -> GND
- C19 pad 1: +3.3V -> +3V3
- C19 pad 2: +5V -> GND
- C20 pad 1: +5V -> GND
- C21 pad 1: +5V -> GND
- C22 pad 1: +5V -> GND
- C24 pad 1: +5V -> GND
- C25 pad 1: +5V -> GND
- C26 pad 1: +5V -> GND
- C27 pad 1: +5V -> GND
- C30 pad 2: +5V -> GND
- C31 pad 2: +5V -> GND
- C32 pad 2: +5V -> GND
- C36 pad 1: +5V -> GND
- C36 pad 2: +3.3V -> +3V3
- C37 pad 1: +3.3V -> +3V3
- C37 pad 2: +5V -> GND
- C38 pad 2: +5V -> GND
- C39 pad 1: +5V -> GND
- C41 pad 1: +5V -> GND
- C41 pad 2: +3.3V -> +3V3
- C42 pad 1: +5V -> GND
- C42 pad 2: +2V5 -> +IO2V5
- C43 pad 1: +5V -> GND
- C44 pad 1: +5V -> GND
- C45 pad 1: +5V -> GND
- C46 pad 1: +5V -> GND
- C47 pad 1: +5V -> GND
- C49 pad 2: Net-(J5-Pin_4) -> Net-(J5-Pin_2)
- C50 pad 2: Net-(J5-Pin_5) -> Net-(J5-Pin_6)
- C51 pad 2: Net-(J5-Pin_6) -> Net-(J5-Pin_5)
- C7 pad 2: +5V -> GND
- J1 pad 1: +5V -> GND
- J2 pad 3: +5V -> GND
- J2 pad 6: +5V -> GND
- J2 pad G1: +5V -> GND
- J2 pad G2: +5V -> GND
- J3 pad A1_B12: +5V -> GND
- J3 pad B1_A12: +5V -> GND
- J3 pad SH1: +5V -> GND
- J3 pad SH2: +5V -> GND
- J3 pad SH3: +5V -> GND
- J3 pad SH4: +5V -> GND
- J4 pad A1_B12: +5V -> GND
- J4 pad B1_A12: +5V -> GND
- J4 pad SH1: +5V -> GND
- J4 pad SH2: +5V -> GND
- J4 pad SH3: +5V -> GND
- J4 pad SH4: +5V -> GND
- J5 pad 1: Net-(J5-Pin_1) -> GNDA
- J5 pad 7: GNDA -> Net-(J5-Pin_7)
- J6 pad 1: Net-(J6-Pin_1) -> GNDA
- J6 pad 5: GNDA -> Net-(J6-Pin_5)
- J7 pad 1: /ESP_IO45 -> /ESP_IO9
- J7 pad 2: /ESP_IO46 -> +3V3
- J7 pad 3: /ESP_IO47 -> /ESP_IO10
- J7 pad 4: /ESP_IO48 -> /ESP_IO13
- J7 pad 5: /ESP_IO40 -> /ESP_IO11
- J7 pad 6: /ESP_IO41 -> /ESP_IO14
- J7 pad 7: /ESP_IO42 -> /ESP_IO12
- J7 pad 8: +5V -> /ESP_IO15
- LED1 pad 2: +3.3V -> +3V3
- MP1 pad 1: +5V -> GND
- Q1 pad 1: +5V -> GND
- Q1 pad 3: /~{USB_RST} -> /~{DBG_RST}
- Q1 pad 4: +5V -> GND
- Q1 pad 5: /~{DBG_ACT} -> Net-(Q1A-D)
- Q1 pad 6: /~{DBG_ACT} -> Net-(Q1A-D)
- R1 pad 1: /HDMI_SCL -> Net-(U11-OUT)
- R1 pad 2: +3.3V -> Net-(U15-B2)
- R11 pad 1: +5V -> GND
- R12 pad 1: +5V -> GND
- R13 pad 1: +5V -> GND
- R2 pad 1: /HDMI_SDA -> Net-(U11-OUT)
- R2 pad 2: +3.3V -> Net-(U15-B3)
- R25 pad 2: unconnected-(R25-Pad2) -> GND
- R26 pad 1: +3.3V -> +3V3
- R36 pad 1: +3.3V -> +3V3
- R37 pad 1: /~{DBG_ACT} -> Net-(Q1A-D)
- R38 pad 1: /~{USB_RST} -> /~{DBG_RST}
- R43 pad 1: /ESP_IO35/GP0 -> Net-(U7-GP0)
- R43 pad 2: Net-(U7-GP0) -> /ESP_IO35/GP0
- R44 pad 1: /ESP_IO36/GP1 -> Net-(U7-GP1)
- R44 pad 2: Net-(U7-GP1) -> /ESP_IO36/GP1
- R45 pad 1: Net-(LED1-K) -> /HDDLED
- R45 pad 2: /HDDLED -> Net-(LED1-K)
- R46 pad 1: Net-(J4-CC1) -> GND
- R46 pad 2: +5V -> Net-(J4-CC1)
- R47 pad 1: Net-(J4-CC2) -> GND
- R47 pad 2: +5V -> Net-(J4-CC2)
- R48 pad 1: Net-(J3-CC1) -> GND
- R48 pad 2: +5V -> Net-(J3-CC1)
- R49 pad 1: Net-(J3-CC2) -> GND
- R49 pad 2: +5V -> Net-(J3-CC2)
- R50 pad 2: +5V -> +3V3
- R72 pad 1: /~{SLT_WAIT} -> GND
- R72 pad 2: +5V -> /~{SLT_WAIT}
- R99 pad 1: +5V -> GND
- S1 pad 2: +5V -> GND
- S3 pad 2: +5V -> GND
- U1 pad 100: /ESP_IO39 -> /ESP_IO38/GP3
- U1 pad 11: +3.3V -> +3V3
- U1 pad 121: +5V -> GND
- U1 pad 122: +5V -> GND
- U1 pad 123: +5V -> GND
- U1 pad 124: +5V -> GND
- U1 pad 13: +3.3V -> +3V3
- U1 pad 15: +3.3V -> +3V3
- U1 pad 2: +5V -> GND
- U1 pad 23: /~{SLT_WAIT} -> /~{SLT_RFSH}
- U1 pad 29: /~{SLT_RFSH} -> /~{SLT_WAIT}
- U1 pad 4: +5V -> GND
- U1 pad 40: /HDMI_SDA -> /SD_DAT3
- U1 pad 42: /HDMI_SCL -> /SD_DAT2
- U1 pad 44: /CODEC_MCK -> /SD_CMD
- U1 pad 46: /CODEC_BCK -> /SD_CD
- U1 pad 48: /CODEC_FS -> /SD_CLK
- U1 pad 50: /CODEC_DACIN -> /SD_DAT0
- U1 pad 52: /CODEC_ADCOUT -> /SD_DAT1
- U1 pad 54: /CODEC_SCLK -> /SD_WP
- U1 pad 56: /CODEC_SDIO -> /~{HDMI_EN}
- U1 pad 6: +5V -> GND
- U1 pad 60: /CODEC_MODE -> /CODEC_SCLK
- U1 pad 61: /SLT_Y1 -> /CODEC_FS
- U1 pad 62: /ESP_IO21/USBEN -> /CODEC_MCK
- U1 pad 63: /SLT_Y0 -> /SLT_Y1
- U1 pad 64: /SD_CLK -> /CODEC_SDIO
- U1 pad 65: /DBG_RXD -> /SLT_Y0
- U1 pad 66: /SD_CMD -> /CODEC_MODE
- U1 pad 67: /DBG_TXD -> /CODEC_BCK
- U1 pad 68: /SD_DAT0 -> /HDMI_SDA
- U1 pad 69: /~{DBG_ACT} -> /CODEC_ADCOUT
- U1 pad 70: /SD_DAT1 -> /HDMI_SCL
- U1 pad 71: /PUSH_BUTTON -> /CODEC_DACIN
- U1 pad 72: /SD_DAT2 -> /HDMI_CEC
- U1 pad 74: /SD_DAT3 -> /HDMI_HPD
- U1 pad 76: /SD_WP -> /DBG_TXD
- U1 pad 78: /SD_CD -> /DBG_RXD
- U1 pad 79: /SND2 -> /ESP_TXD
- U1 pad 8: +5V -> GND
- U1 pad 80: /DBG_SCL -> /~{DBG_RST}
- U1 pad 81: /SND1 -> /PUSH_BUTTON
- U1 pad 82: /DBG_SDA -> /ESP_EN
- U1 pad 83: /SND0 -> /SND2
- U1 pad 84: /ESP_TXD -> /ESP_RXD
- U1 pad 85: /ESP_EN -> /SND1
- U1 pad 86: /ESP_RXD -> /ESP_IO21/USBEN
- U1 pad 87: /ESP_BOOT_MODE -> /SND0
- U1 pad 88: /ESP_IO17/SCL -> /ESP_BOOT_MODE
- U1 pad 9: +3.3V -> +3V3
- U1 pad 90: /ESP_IO18/SDA -> /ESP_IO17/SCL
- U1 pad 92: /ESP_IO35/GP0 -> /ESP_IO18/SDA
- U1 pad 94: /ESP_IO36/GP1 -> /ESP_IO35/GP0
- U1 pad 96: /ESP_IO37/GP2 -> /ESP_IO36/GP1
- U1 pad 98: /ESP_IO38/GP3 -> /ESP_IO37/GP2
- U10 pad 3: +5V -> GND
- U12 pad 11: +5V -> GND
- U14 pad 10: +2V5 -> +IO2V5
- U14 pad 11: +5V -> GND
- U14 pad 2: +2V5 -> +IO2V5
- U2 pad 10: +5V -> GND
- U3 pad 10: +5V -> GND
- U4 pad 12: +5V -> /~{HDMI_EN}
- U4 pad 13: +5V -> GND
- U4 pad 16: +5V -> GND
- U4 pad 20: +5V -> GND
- U4 pad 21: +5V -> GND
- U4 pad 25: +5V -> GND
- U4 pad 28: +5V -> GND
- U4 pad 29: +3.3V -> +3V3
- U4 pad 32: +3.3V -> +3V3
- U4 pad 4: +3.3V -> +3V3
- U4 pad 5: +3.3V -> +3V3
- U4 pad 9: +3.3V -> +3V3
- U5 pad 23: Net-(J6-Pin_3) -> Net-(J6-Pin_4)
- U5 pad 24: +5V -> GND
- U5 pad 25: Net-(J6-Pin_4) -> Net-(J6-Pin_5)
- U5 pad 28: +5V -> GND
- U5 pad 29: Net-(J6-Pin_2) -> Net-(J6-Pin_3)
- U5 pad 3: Net-(J5-Pin_1) -> Net-(J5-Pin_4)
- U5 pad 30: Net-(J6-Pin_1) -> Net-(J6-Pin_2)
- U5 pad 33: +5V -> GND
- U5 pad 6: Net-(J5-Pin_2) -> Net-(J5-Pin_7)
- U6 pad 1: +5V -> GND
- U6 pad 16: /ESP_IO46 -> unconnected-(U6-IO46-Pad16)
- U6 pad 2: +3.3V -> +3V3
- U6 pad 24: /ESP_IO47 -> unconnected-(U6-IO47-Pad24)
- U6 pad 25: /ESP_IO48 -> unconnected-(U6-IO48-Pad25)
- U6 pad 26: /ESP_IO45 -> unconnected-(U6-IO45-Pad26)
- U6 pad 32: /ESP_IO39 -> unconnected-(U6-IO39-Pad32)
- U6 pad 33: /ESP_IO40 -> unconnected-(U6-IO40-Pad33)
- U6 pad 34: /ESP_IO41 -> unconnected-(U6-IO41-Pad34)
- U6 pad 35: /ESP_IO42 -> unconnected-(U6-IO42-Pad35)
- U6 pad 40: +5V -> GND
- U6 pad 41: +5V -> GND
- U7 pad 14: +5V -> GND
- U7 pad 4: /~{USB_RST} -> /~{DBG_RST}
- U8 pad 10: +5V -> GND
- U9 pad 1: /USB_VBUS -> /ESP_IO21/USBEN
- U9 pad 2: +5V -> GND
- U9 pad 4: /ESP_IO21/USBEN -> +5V
- U9 pad 5: +5V -> /USB_VBUS
- X1 pad 41: +5V -> GND
- X1 pad 43: +5V -> GND
- X2 pad 11: +5V -> GND
- X2 pad 13: unconnected-(X2-CEC-Pad13) -> Net-(U15-B1)
- X2 pad 15: /HDMI_SCL -> Net-(U15-B2)
- X2 pad 16: /HDMI_SDA -> Net-(U15-B3)
- X2 pad 17: +5V -> GND
- X2 pad 18: +5V -> Net-(U11-OUT)
- X2 pad 19: unconnected-(X2-HPD-Pad19) -> Net-(U15-B4)
- X2 pad 2: +5V -> GND
- X2 pad 5: +5V -> GND
- X2 pad 8: +5V -> GND
- X2 pad S1: +5V -> GND
- X2 pad S2: +5V -> GND
- X2 pad S3: +5V -> GND
- X2 pad S4: +5V -> GND
- X3 pad 10: +5V -> GND
- X3 pad 2: +5V -> GND
Routing:
- net GND: track 0.00 -> 165.1 mm, vias 0 -> 7
- net (no net): track 90.4 -> 0.05 mm
- net GNDA: track 50.7 -> 114.2 mm, vias 0 -> 1
- net /TDI: track 0.00 -> 56.3 mm
- net /TMS: track 0.00 -> 55.6 mm
- net /CODEC_FS: track 0.00 -> 54.5 mm, vias 0 -> 2
- net /CODEC_BCK: track 0.00 -> 54.1 mm, vias 0 -> 2
- net /TDO: track 0.00 -> 53.8 mm
- net /CODEC_ADCOUT: track 0.00 -> 53.3 mm, vias 0 -> 2
- net /CODEC_DACIN: track 0.00 -> 53.1 mm, vias 0 -> 2
- net /CODEC_MCK: track 0.00 -> 50.0 mm, vias 0 -> 2
- net /TCK: track 0.00 -> 48.6 mm, vias 0 -> 2
- net /JTAGVCC: track 0.00 -> 48.3 mm
- net /CODEC_MODE: track 0.00 -> 47.0 mm, vias 0 -> 2
- net /CODEC_SDIO: track 0.00 -> 45.6 mm, vias 0 -> 2
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Other:
- board size 99 x 65.6 mm -> 99.6 x 65.6 mm

Commit message: PCB work in progress
Parts:
- added FL1: DLM0NSN900HY2D, Library:FIL_DLM0NSN900HY2D, B.Cu at (178.0, 78.7)
- J3: moved to B.Cu
- moved R50 46.6 mm to (169.9, 82.4), turned to -90 degrees
- moved C27 42.7 mm to (173.3, 85.0)
- moved U9 41.9 mm to (173.2, 82.3)
- moved C41 19.6 mm to (183.9, 118.5)
- moved C37 18.9 mm to (188.3, 114.4)
- moved C36 17.0 mm to (190.1, 117.3)
- moved R99 14.8 mm to (111.7, 108.5)
- moved R44 13.5 mm to (179.0, 92.3)
- moved R43 13.2 mm to (179.1, 90.3)
- moved J7 10.5 mm to (183.7, 90.0)
- moved R37 10.1 mm to (192.1, 82.1), turned to -90 degrees
- moved C25 9.47 mm to (181.9, 77.9), turned to 180 degrees
- moved R40 8.36 mm to (166.1, 71.3), turned to 0 degrees
- moved Q1 7.65 mm to (189.4, 81.7), turned to 0 degrees
- moved C54 7.00 mm to (174.8, 78.8), turned to -90 degrees
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Connections:
- J3 pad A6: /ESP_USB_Dp -> Net-(J3-DP1)
- J3 pad A7: /ESP_USB_Dn -> Net-(J3-DN1)
- J3 pad B6: /ESP_USB_Dp -> Net-(J3-DP1)
- J3 pad B7: /ESP_USB_Dn -> Net-(J3-DN1)
- R40 pad 1: Net-(U15-B4) -> Net-(U15-B1)
- U1 pad 100: /ESP_IO38/GP3 -> /ESP_IO14
- U1 pad 101: /ESP_IO7 -> /ESP_IO15
- U1 pad 102: /ESP_IO11 -> /ESP_IO13
- U1 pad 105: /ESP_IO9 -> /ESP_IO18/SDA
- U1 pad 106: /ESP_IO13 -> /ESP_IO11
- U1 pad 107: /ESP_IO10 -> /ESP_IO17/SCL
- U1 pad 108: /ESP_IO14 -> /ESP_IO10
- U1 pad 110: /ESP_IO15 -> /ESP_IO9
- U1 pad 112: /ESP_IO16 -> /ESP_EN
- U1 pad 66: /CODEC_MODE -> /ESP_BOOT_MODE
- U1 pad 68: /HDMI_SDA -> /CODEC_MODE
- U1 pad 70: /HDMI_SCL -> /HDMI_CEC
- U1 pad 72: /HDMI_CEC -> /HDMI_SCL
- U1 pad 74: /HDMI_HPD -> /HDMI_SDA
- U1 pad 76: /DBG_TXD -> /HDMI_HPD
- U1 pad 78: /DBG_RXD -> /~{DBG_RST}
- U1 pad 79: /ESP_TXD -> /DBG_TXD
- U1 pad 80: /~{DBG_RST} -> /DBG_RXD
- U1 pad 82: /ESP_EN -> /ESP_IO35/GP0
- U1 pad 84: /ESP_RXD -> /ESP_IO36/GP1
- U1 pad 86: /ESP_IO21/USBEN -> /ESP_IO37/GP2
- U1 pad 88: /ESP_BOOT_MODE -> /ESP_IO38/GP3
- U1 pad 89: /ESP_IO1 -> /ESP_IO16
- U1 pad 90: /ESP_IO17/SCL -> /ESP_RXD
- U1 pad 91: /ESP_IO2 -> /ESP_IO3
- U1 pad 92: /ESP_IO18/SDA -> /ESP_TXD
- U1 pad 93: /ESP_IO3 -> /ESP_IO4
- U1 pad 94: /ESP_IO35/GP0 -> /ESP_IO2
- U1 pad 95: /ESP_IO4 -> /ESP_IO5
- U1 pad 96: /ESP_IO36/GP1 -> /ESP_IO1
- U1 pad 97: /ESP_IO5 -> /ESP_IO6
- U1 pad 98: /ESP_IO37/GP2 -> /ESP_IO21/USBEN
- U1 pad 99: /ESP_IO6 -> /ESP_IO7
- U15 pad 2: /HDMI_CEC -> /HDMI_HPD
- U15 pad 3: /HDMI_SCL -> /HDMI_SDA
- U15 pad 4: /HDMI_SDA -> /HDMI_SCL
- U15 pad 5: /HDMI_HPD -> /HDMI_CEC
- X2 pad 13: Net-(U15-B1) -> Net-(U15-B4)
- X2 pad 15: Net-(U15-B2) -> Net-(U15-B3)
- X2 pad 16: Net-(U15-B3) -> Net-(U15-B2)
- X2 pad 19: Net-(U15-B4) -> Net-(U15-B1)
Routing:
- net Net-(C18-Pad2): track 0.00 -> 146.8 mm, vias 0 -> 2
- net /ESP_IO17/SCL: track 0.00 -> 88.2 mm, vias 0 -> 5
- net /ESP_IO18/SDA: track 0.00 -> 84.6 mm, vias 0 -> 5
- net /~{DBG_RST}: track 0.00 -> 81.4 mm, vias 0 -> 2
- net /ESP_IO38/GP3: track 0.00 -> 68.6 mm, vias 0 -> 3
- net /DBG_TXD: track 0.00 -> 66.7 mm, vias 0 -> 3
- net /PUSH_BUTTON: track 0.00 -> 65.5 mm, vias 0 -> 4
- net /DBG_RXD: track 0.00 -> 65.3 mm, vias 0 -> 1
- net /ESP_BOOT_MODE: track 0.00 -> 60.5 mm, vias 0 -> 2
- net /ESP_IO37/GP2: track 0.00 -> 51.7 mm, vias 0 -> 2
- net /~{HDMI_EN}: track 35.3 -> 74.4 mm
- net /HDMI_HPD: track 0.00 -> 37.9 mm, vias 0 -> 1
- net /HDMI_SDA: track 0.00 -> 36.9 mm, vias 0 -> 1
- net /ESP_IO1: track 0.00 -> 36.4 mm, vias 0 -> 1
- net /HDMI_SCL: track 0.00 -> 36.4 mm, vias 0 -> 1
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Other:
- board size 99.6 x 65.6 mm -> 99 x 65.6 mm

Commit message: PCB work in progress
Parts:
- added FL2: DLM0NSN900HY2D, Library:FIL_DLM0NSN900HY2D, F.Cu at (186.5, 74.5)
- C24, C52, C53, C54, R48, R49, U11, U7: moved to F.Cu
- C27, R13, R46, R47, R50, U9: moved to B.Cu
- moved R13 18.0 mm to (144.7, 101.8), turned to 90 degrees
- moved C53 15.3 mm to (167.2, 81.7), turned to 0 degrees
- moved R50 15.0 mm to (184.9, 82.8), turned to 180 degrees
- moved C41 13.2 mm to (185.8, 105.4), turned to 180 degrees
- moved U11 12.2 mm to (167.8, 84.3), turned to 0 degrees
- moved U9 12.1 mm to (185.0, 79.6), turned to 90 degrees
- moved C36 11.2 mm to (185.8, 107.0)
- moved C52 11.2 mm to (167.2, 87.0), turned to 0 degrees
- moved C27 9.57 mm to (182.4, 82.1), turned to -90 degrees
- moved U7 9.49 mm to (181.7, 81.6)
- moved C24 9.36 mm to (176.3, 78.6)
- moved R11 8.86 mm to (182.9, 106.2), turned to -90 degrees
- moved C54 7.72 mm to (167.2, 80.1), turned to 0 degrees
- moved C37 6.37 mm to (185.8, 108.6), turned to 0 degrees
- moved R47 6.23 mm to (191.6, 73.5)
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Connections:
- J4 pad A6: /DBG_Dp -> Net-(J4-DP1)
- J4 pad A7: /DBG_Dn -> Net-(J4-DN1)
- J4 pad B6: /DBG_Dp -> Net-(J4-DP1)
- J4 pad B7: /DBG_Dn -> Net-(J4-DN1)
- J7 pad 1: /ESP_IO9 -> /ESP_IO2
- J7 pad 10: /ESP_IO16 -> /ESP_IO9
- J7 pad 3: /ESP_IO10 -> /ESP_IO14
- J7 pad 4: /ESP_IO13 -> /ESP_IO1
- J7 pad 5: /ESP_IO11 -> /ESP_IO12
- J7 pad 6: /ESP_IO14 -> /ESP_IO13
- J7 pad 7: /ESP_IO12 -> /ESP_IO10
- J7 pad 8: /ESP_IO15 -> /ESP_IO11
Routing:
- net +5V: track 75.9 -> 177.6 mm, vias 5 -> 7
- net +IO1V8: track 1.63 -> 90.8 mm, vias 0 -> 4
- net GND: track 196.1 -> 247.4 mm, vias 7 -> 8
- net /ESP_IO9: track 14.7 -> 48.2 mm
- net /ESP_IO21/USBEN: track 24.5 -> 58.0 mm, vias 1 -> 2
- net /ESP_IO11: track 15.1 -> 46.5 mm
- net /ESP_BOOT_MODE: track 60.5 -> 91.1 mm, vias 2 -> 3
- net /ESP_IO10: track 14.9 -> 44.3 mm
- net /ESP_IO12: track 19.4 -> 45.7 mm
- net /ESP_IO13: track 25.2 -> 48.7 mm
- net +IO2V5: track 9.68 -> 29.1 mm, vias 2 -> 4
- net /USB_VBUS: track 0.01 -> 17.8 mm
- net /ESP_IO17/SCL: track 88.2 -> 71.6 mm, vias 5 -> 4
- net /ESP_IO14: track 29.8 -> 46.1 mm
- net /ESP_IO1: track 36.4 -> 51.3 mm
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Other:
- board size 99 x 65.6 mm -> 102 x 65.5 mm

Commit message: PCB work in progress
Parts:
- C1: moved to B.Cu
- J1: value Conn_01x02_Pin -> Conn_01x03; footprint Library:JUMPER_1 -> Connector_PinHeader_2.54mm:PinHeader_1x03_P2.54mm_Vertical
- U1: value SOM_FPGA_LP -> CONN_DF40C-120DP-0p4V51_120P_HIR
- moved R99 12.3 mm to (99.3, 107.7)
- moved J1 6.41 mm to (130.9, 108.7), turned to 0 degrees
- moved C30 4.36 mm to (133.6, 108.5), turned to 90 degrees
- moved VR1 3.55 mm to (103.8, 106.8), turned to 0 degrees
- moved C22 2.69 mm to (106.7, 107.0), turned to 90 degrees
- moved R72 2.63 mm to (168.8, 119.6)
- moved C32 1.45 mm to (103.2, 109.3)
- moved C1 1.15 mm to (123.9, 123.2), turned to 180 degrees
- moved R50 1.14 mm to (185.9, 83.3), turned to -90 degrees
- moved C29 1.00 mm to (104.3, 92.3)
- moved C39 1.00 mm to (105.8, 92.3)
- moved R29 0.94 mm to (132.8, 101.2), turned to 180 degrees
- moved C11 0.86 mm to (138.9, 108.5), turned to -90 degrees
- moved C20 0.86 mm to (136.7, 108.5), turned to -90 degrees
- moved C44 0.86 mm to (135.2, 108.5), turned to -90 degrees
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Routing:
- net GND: track 247.4 -> 776.0 mm, vias 8 -> 22
- net +3V3: track 88.6 -> 339.5 mm, vias 5 -> 17
- net +5V: track 177.6 -> 232.8 mm, vias 7 -> 11
- net GNDA: track 101.1 -> 129.3 mm, vias 1 -> 4
- net +3V3DAC: track 4.42 -> 30.2 mm, vias 0 -> 3
- net +IO3V3: track 0.00 -> 10.4 mm, vias 0 -> 2
- net +IO1V8: track 90.8 -> 84.3 mm
- net /~{DBG_RST}: track 71.1 -> 66.6 mm
- net /ESP_BOOT_MODE: track 91.1 -> 95.5 mm
- net Net-(C18-Pad2): track 146.8 -> 151.0 mm
- net +IO2V5: track 29.1 -> 32.9 mm
- net Net-(R19-Pad1): track 0.00 -> 3.70 mm
- net Net-(R17-Pad1): track 0.00 -> 3.70 mm
- net Net-(R18-Pad1): track 0.00 -> 3.70 mm
- net Net-(R16-Pad1): track 0.00 -> 3.70 mm
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Other:
- board text added: "3V3"
- board text added: "5V"
- board text added: "GND"
- board text removed: "+"
- board text removed: "+5V"
