File: board/HyperFusionXC.kicad_sch (KiCad schematic)
At the start: 103 parts, among them J1 Conn_01x02_Pin, U1 10CL025YE144C8G, U10 SN74LVC1G04DCKR, U12 TXS0108EPWR, U14 TXS0108EPWR, U2 74AHC541, U3 74AHC541, U4 M25P80-VMN3TPB, U5 PCM5101APWR, U6 AT93C46DN-SH-T, U7 SG3225CAN 50.0000M-TJGA6, U8 74AHC541, U9 PCM1808PWR, X1 EDGE50/MSX, X3 302-S101

Commit message: Work in progress
Parts:
- added C16, C17, C45: 100nF, Capacitor_SMD:C_0603_1608Metric, symbol Sheet1-altium-import:root_1_C_0805
Connections:
- net +3V3: now also U10.5 (VCC), C16.1, C17.1, C45.1
- net EDGE_A0: now also U3.5 (A3); no longer U3.4 (A2)
- net EDGE_A1: now also U3.4 (A2); no longer U3.5 (A3)
- net EDGE_A2: now also U3.7 (A5); no longer U3.6 (A4)
- net EDGE_A3: now also U3.6 (A4); no longer U3.7 (A5)
- net EDGE_A4: now also U3.9 (A7); no longer U3.8 (A6)
- net EDGE_A5: now also U3.8 (A6); no longer U3.9 (A7)
- net EDGE_A6: now also U3.3 (A1); no longer U3.2 (A0)
- net EDGE_A7: now also U3.2 (A0); no longer U3.3 (A1)
- net EDGE_CLC: now also U14.18 (B2); no longer U14.12 (B8)
- net GND: now also U1.22 (CLK0), U10.3 (GND), C16.2, C17.2, C45.2; no longer U1.88 (CLK7)
- net SLT_CLC: now also U1.88 (CLK7), U14.3 (A2); no longer U1.22 (CLK0), U14.9 (A8)
- net SLT_X0: now also U3.17 (Y1); no longer U3.18 (Y0)
- net SLT_X1: now also U3.18 (Y0); no longer U3.17 (Y1)
- net SLT_X2: now also U3.15 (Y3); no longer U3.16 (Y2)
- net SLT_X3: now also U3.16 (Y2); no longer U3.15 (Y3)
- net SLT_X4: now also U3.13 (Y5); no longer U3.14 (Y4)
- net SLT_X5: now also U3.14 (Y4); no longer U3.13 (Y5)
- net SLT_X6: now also U3.11 (Y7); no longer U3.12 (Y6)
- net SLT_X7: now also U3.12 (Y6); no longer U3.11 (Y7)
- net SLT_Y0: now also U1.59 (IO_21); no longer U1.65 (IO_23)
- net SLT_Y1: now also U1.65 (IO_23); no longer U1.60 (IO_22)
- net SLT_Y2: now also U1.60 (IO_22); no longer U1.59 (IO_21)
- net SLT_Y3: now also U1.66 (IO_24); no longer U1.58 (IO_20)
- net ~{EDGE_BUSDIR}: now also U14.13 (B7); no longer U14.15 (B5)
- net ~{EDGE_CS1}: now also U8.3 (A1); no longer U8.2 (A0)
- net ~{EDGE_CS2}: now also U8.2 (A0); no longer U8.3 (A1)
- net ~{EDGE_INT}: now also U14.14 (B6); no longer U14.16 (B4)
- net ~{EDGE_RESET}: now also U14.12 (B8); no longer U14.14 (B6)
- net ~{EDGE_RFSH}: now also U14.16 (B4); no longer U14.18 (B2)
- net ~{EDGE_SLTSEL}: now also U14.17 (B3); no longer U14.20 (B1)
- net ~{EDGE_WAIT}: now also U14.15 (B5); no longer U14.17 (B3)
- net ~{SLT_BUSDIR}: now also U1.71 (IO_28), U14.8 (A7); no longer U1.72 (IO_29), U14.6 (A5)
- net ~{SLT_INT}: now also U1.72 (IO_29), U14.7 (A6); no longer U1.71 (IO_28), U14.5 (A4)
- net ~{SLT_RESET}: now also U1.69 (IO_27), U14.9 (A8); no longer U1.76 (IO_30), U14.7 (A6)
- net ~{SLT_RFSH}: now also U1.67 (IO_25), U14.5 (A4); no longer U1.68 (IO_26), U14.3 (A2)
- net ~{SLT_SLTSL}: now also U1.76 (IO_30), U14.4 (A3); no longer U1.67 (IO_25), U14.1 (A1)
- net ~{SLT_WAIT}: now also U1.68 (IO_26), U14.6 (A5); no longer U1.69 (IO_27), U14.4 (A3)
- net SLT_SW renamed SLT_MUX
- net SLT_MUX: now also U1.58 (IO_20); no longer U1.66 (IO_24)
- net ~{SLT_SW} renamed ~{SLT_MUX}

Commit message: Work in progress
Connections:
- net ADC_BCK: now also U1.141 (IO_58); no longer U1.142 (IO_59)
- net ADC_DOUT: now also U1.22 (CLK0); no longer U1.141 (IO_58)
- net ADC_LRCK: now also U1.142 (IO_59); no longer U1.144 (IO_61)
- net DAC_BCK: now also U1.11 (IO_5), U1.31 (IO_9); no longer U1.28 (IO_8)
- net DAC_DIN: now also U1.10 (IO_4); no longer U1.11 (IO_5)
- net DAC_FLT: now also U1.33 (IO_11); no longer U1.32 (IO_10)
- net DAC_LRCK: now also U1.7 (IO_2); no longer U1.10 (IO_4)
- net DAC_SCK: now also U1.28 (IO_8), U1.32 (IO_10); no longer U1.31 (IO_9)
- net DAC_XSMT: now also U1.144 (IO_61); no longer U1.7 (IO_2)
- net GND: now also U5.10 (DEMP), U9.10 (MD0), U9.11 (MD1); no longer U1.22 (CLK0)
- net TCK: now also U1.16 (TCK)
- net TDI: now also U1.15 (TDI)
- net TDO: now also U1.20 (TDO)
- net TMS: now also U1.18 (TMS)
- net ADC_MD0: no longer names the net of U1.137 (IO_57)
- net ADC_MD0: no longer U9.10 (MD0)
- net ADC_MD1: no longer names the net of U1.136 (IO_56)
- net ADC_MD1: no longer U9.11 (MD1)
- removed net DAC_DEMP: U1.33 (IO_11), U5.10 (DEMP)
Changed lines of the file:
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@@
 	)
 	(junction
+		(at 414.02 76.2)
+		(diameter 0)
+		(color 0 0 0 0)
+	)
+	(junction
 		(at 410.21 306.07)
 		(diameter 0)
@@
 	)
 	(junction
+		(at 264.16 88.9)
+		(diameter 0)
+		(color 0 0 0 0)
+	)
+	(junction
 		(at 331.47 344.17)
 		(diameter 0)
@@
 	)
 	(junction
+		(at 264.16 86.36)
+		(diameter 0)
+		(color 0 0 0 0)
+	)
+	(junction
 		(at 388.62 195.58)
 		(diameter 0)
@@
 	(wire
 		(pts
-			(xy 426.72 60.96) (xy 434.34 60.96)
+			(xy 127 48.26) (xy 128.27 48.26)
 		)
 		(stroke
@@
 	(wire
 		(pts
-			(xy 127 48.26) (xy 128.27 48.26)
+			(xy 492.76 69.85) (xy 499.11 69.85)
 		)
 		(stroke
@@
 	(wire
 		(pts
-			(xy 492.76 69.85) (xy 499.11 69.85)
+			(xy 513.08 289.56) (xy 516.89 289.56)
 		)
 		(stroke
@@
 	(wire
 		(pts
-			(xy 513.08 289.56) (xy 516.89 289.56)
+			(xy 481.33 80.01) (xy 482.6 80.01)
 		)
 		(stroke
@@
 	(wire
 		(pts
-			(xy 481.33 80.01) (xy 482.6 80.01)
+			(xy 372.11 196.85) (xy 372.11 195.58)
 		)
 		(stroke
@@
 	(wire
 		(pts
-			(xy 372.11 196.85) (xy 372.11 195.58)
+			(xy 264.16 83.82) (xy 264.16 86.36)
 		)
 		(stroke
@@
 	(wire
 		(pts
+			(xy 265.43 83.82) (xy 264.16 83.82)
+		)
+		(stroke
+			(width 0)
+			(type default)
+		)
+	)
+	(wire
+		(pts
 			(xy 212.09 236.22) (xy 212.09 234.95)
 		)
@@
 	(wire
 		(pts
-			(xy 257.81 83.82) (xy 265.43 83.82)
-		)
-		(stroke
-			(width 0)
-			(type default)
-		)
-	)
-	(wire
-		(pts
 			(xy 430.53 101.6) (xy 430.53 107.95)
 		)
@@
 	(wire
 		(pts
+			(xy 265.43 86.36) (xy 264.16 86.36)
+		)
+		(stroke
+			(width 0)
+			(type default)
+		)
+	)
+	(wire
+		(pts
 			(xy 298.45 196.85) (xy 298.45 179.07)
 		)
@@
 	(wire
 		(pts
-			(xy 255.27 273.05) (xy 255.27 275.59)
-		)
-		(stroke
-			(width 0)
-			(type default)
-		)
-	)
-	(wire
-		(pts
 			(xy 562.61 341.63) (xy 562.61 345.44)
 		)
@@
 	(wire
 		(pts
+			(xy 264.16 86.36) (xy 264.16 88.9)
+		)
+		(stroke
+			(width 0)
+			(type default)
+		)
+	)
+	(wire
+		(pts
 			(xy 388.62 184.15) (xy 388.62 185.42)
 		)
@@
 	(wire
 		(pts
-			(xy 257.81 273.05) (xy 255.27 273.05)
-		)
-		(stroke
-			(width 0)
-			(type default)
-		)
-	)
-	(wire
-		(pts
 			(xy 354.33 171.45) (xy 359.41 171.45)
 		)
@@
 	(wire
 		(pts
-			(xy 257.81 86.36) (xy 265.43 86.36)
-		)
-		(stroke
-			(width 0)
-			(type default)
-		)
-	)
-	(wire
-		(pts
 			(xy 288.29 349.25) (xy 302.26 349.25)
 		)
@@
 	(wire
 		(pts
+			(xy 414.02 60.96) (xy 414.02 76.2)
+		)
+		(stroke
+			(width 0)
+			(type default)
+		)
+	)
+	(wire
+		(pts
 			(xy 242.57 308.61) (xy 242.57 312.42)
 		)
@@
 	(wire
 		(pts
+			(xy 414.02 60.96) (xy 434.34 60.96)
+		)
+		(stroke
+			(width 0)
+			(type default)
+		)
+	)
+	(wire
+		(pts
 			(xy 538.48 327.66) (xy 538.48 331.47)
 		)
@@
 		)
 	)
-	(hierarchical_label "ADC_MD1"
-		(shape passive)
-		(at 303.53 196.85 90)
-		(effects
-			(font
-				(size 1.27 1.27)
-			)
-			(justify left)
-		)
-	)
 	(hierarchical_label "EDGE_A11"
 		(shape passive)
@@
 		)
 	)
+	(hierarchical_label "TDO"
+		(shape passive)
+		(at 257.81 267.97 180)
+		(effects
+			(font
+				(size 1.27 1.27)
+			)
+			(justify right)
+		)
+	)
 	(hierarchical_label "EDGE_A7"
 		(shape passive)
@@
 		)
 	)
+	(hierarchical_label "TMS"
+		(shape passive)
+		(at 257.81 262.89 180)
+		(effects
+			(font
+				(size 1.27 1.27)
+			)
+			(justify right)
+		)
+	)
 	(hierarchical_label "EDGE_A6"
 		(shape passive)
@@
 		)
 	)
-	(hierarchical_label "ADC_LRCK"
+	(hierarchical_label "DAC_LRCK"
 		(shape passive)
-		(at 283.21 196.85 90)
+		(at 257.81 234.95 180)
 		(effects
 			(font
 				(size 1.27 1.27)
 			)
-			(justify left)
+			(justify right)
 		)
 	)
@@
 		)
 	)
+	(hierarchical_label "TDI"
+		(shape passive)
+		(at 257.81 255.27 180)
+		(effects
+			(font
+				(size 1.27 1.27)
+			)
+			(justify right)
+		)
+	)
 	(hierarchical_label "SLT_X0"
 		(shape passive)
@@
 	(hierarchical_label "ADC_DOUT"
 		(shape passive)
-		(at 290.83 196.85 90)
+		(at 257.81 273.05 180)
 		(effects
 			(font
 				(size 1.27 1.27)
 			)
-			(justify left)
+			(justify right)
 		)
 	)
@@
 	(hierarchical_label "DAC_XSMT"
 		(shape passive)
-		(at 257.81 234.95 180)
+		(at 283.21 196.85 90)
 		(effects
 			(font
 				(size 1.27 1.27)
 			)
-			(justify right)
+			(justify left)
 		)
 	)
@@
 	(hierarchical_label "DAC_FLT"
 		(shape passive)
-		(at 257.81 298.45 180)
+		(at 257.81 300.99 180)
 		(effects
 			(font
@@
 		)
 	)
-	(hierarchical_label "ADC_MD0"
-		(shape passive)
-		(at 300.99 196.85 90)
-		(effects
-			(font
-				(size 1.27 1.27)
-			)
-			(justify left)
-		)
-	)
 	(hierarchical_label "SLT_X7"
 		(shape passive)
@@
 		)
 	)
-	(hierarchical_label "ADC_MD0"
-		(shape passive)
-		(at 257.81 83.82 180)
-		(effects
-			(font
-				(size 1.27 1.27)
-			)
-			(justify right)
-		)
-	)
 	(hierarchical_label "TDI"
 		(shape passive)
@@
 	(hierarchical_label "ADC_BCK"
 		(shape passive)
-		(at 288.29 196.85 90)
+		(at 290.83 196.85 90)
 		(effects
 			(font
@@
 		)
 	)
-	(hierarchical_label "DAC_DEMP"
-		(shape passive)
-		(at 426.72 60.96 180)
-		(effects
-			(font
-				(size 1.27 1.27)
-			)
-			(justify right)
-		)
-	)
 	(hierarchical_label "DAC_BCK"
 		(shape passive)
@@
 	(hierarchical_label "DAC_DIN"
 		(shape passive)
-		(at 257.81 245.11 180)
+		(at 257.81 242.57 180)
 		(effects
 			(font
@@
 		)
 	)
-	(hierarchical_label "ADC_MD1"
-		(shape passive)
-		(at 257.81 86.36 180)
-		(effects
-			(font
-				(size 1.27 1.27)
-			)
-			(justify right)
-		)
-	)
 	(hierarchical_label "EDGE_D2"
 		(shape passive)
@@
 	(hierarchical_label "DAC_SCK"
 		(shape passive)
-		(at 257.81 295.91 180)
+		(at 257.81 298.45 180)
 		(effects
 			(font
@@
 		)
 	)
+	(hierarchical_label "DAC_BCK"
+		(shape passive)
+		(at 257.81 245.11 180)
+		(effects
+			(font
+				(size 1.27 1.27)
+			)
+			(justify right)
+		)
+	)
 	(hierarchical_label "EDGE_D1"
 		(shape passive)
@@
 	(hierarchical_label "DAC_BCK"
 		(shape passive)
-		(at 257.81 288.29 180)
+		(at 257.81 295.91 180)
 		(effects
 			(font
@@
 		)
 	)
-	(hierarchical_label "DAC_DEMP"
-		(shape passive)
-		(at 257.81 300.99 180)
-		(effects
-			(font
-				(size 1.27 1.27)
-			)
-			(justify right)
-		)
-	)
 	(hierarchical_label "~{EDGE_WR}"
 		(shape passive)
@@
 		)
 	)
-	(hierarchical_label "DAC_LRCK"
+	(hierarchical_label "ADC_LRCK"
 		(shape passive)
-		(at 257.81 242.57 180)
+		(at 288.29 196.85 90)
 		(effects
 			(font
 				(size 1.27 1.27)
 			)
-			(justify right)
+			(justify left)
 		)
 	)
@@
 		)
 	)
+	(hierarchical_label "TCK"
+		(shape passive)
+		(at 257.81 257.81 180)
+		(effects
+			(font
+				(size 1.27 1.27)
+			)
+			(justify right)
+		)
+	)
 	(hierarchical_label "SLT_X2"
 		(shape passive)
@@
 		)
 	)
+	(hierarchical_label "DAC_SCK"
+		(shape passive)
+		(at 257.81 288.29 180)
+		(effects
+			(font
+				(size 1.27 1.27)
+			)
+			(justify right)
+		)
+	)

Commit message: Work in progress
Parts:
- removed C10, C8: 100nF, Capacitor_SMD:C_0603_1608Metric, symbol Sheet1-altium-import:root_0_C_0805
- removed C103, C203: 1uF 10V, Capacitor_Tantalum_SMD:CP_EIA-3216-10_Kemet-I_Pad1.58x1.35mm_HandSolder, symbol Sheet1-altium-import:root_0_CAP100RP
- removed C105, C29: 10uF 10V, Capacitor_Tantalum_SMD:CP_EIA-3216-10_Kemet-I_Pad1.58x1.35mm_HandSolder, symbol Sheet1-altium-import:root_0_CAP100RP
- removed C15, C18, C39, C40, C41, C42, C43: 100nF, Capacitor_SMD:C_0603_1608Metric, symbol Sheet1-altium-import:root_1_C_0805
- removed C2, C22, C23, C3: 10uF 10V, Capacitor_Tantalum_SMD:CP_EIA-3216-10_Kemet-I_Pad1.58x1.35mm_HandSolder, symbol Sheet1-altium-import:root_3_CAP100RP
- removed C36: 2.2nF, Capacitor_SMD:C_0603_1608Metric, symbol Sheet1-altium-import:root_1_C_0805
- removed R43, R44, R63, R65, R66, R67, R68, R69: 10E, Resistor_SMD:R_0603_1608Metric, symbol Sheet1-altium-import:root_2_R_0805
- removed R46, R47, R48, R56: 10k, Resistor_SMD:R_0603_1608Metric, symbol Sheet1-altium-import:root_2_R_0805
- removed R49, R60, R61: 470E, Resistor_SMD:R_0603_1608Metric, symbol Sheet1-altium-import:root_2_R_0805
- removed R57, R70, R71: 1k, Resistor_SMD:R_0603_1608Metric, symbol Sheet1-altium-import:root_1_R_0805
- removed R58, R59: 10k, Resistor_SMD:R_0603_1608Metric, symbol Sheet1-altium-import:root_1_R_0805
- removed R62: 25E, Resistor_SMD:R_0603_1608Metric, symbol Sheet1-altium-import:root_1_R_0805
- removed TP1: TestPoint, Library:TestPoint_THTPad_D1.5mm_Drill0.9mm, symbol Connector:TestPoint
- removed U1: 10CL025YE144C8G, Library:QFP50P2200X2200X165-145N, symbol Library:10CL025YE144C8G
- removed U4: M25P80-VMN3TPB, Package_SO:SO-8_3.9x4.9mm_P1.27mm, symbol Library:M25P80-VMN
- removed U6: AT93C46DN-SH-T, Package_SO:SO-8_3.9x4.9mm_P1.27mm, symbol Library:AT93C46DN
- removed U7: SG3225CAN 50.0000M-TJGA6, Library:SG3225CAN, symbol Sheet1-altium-import:root_0_SG-310
- removed UCT1: AP2114HA-1.2TRG1, Package_TO_SOT_SMD:SOT-223, symbol Sheet1-altium-import:root_0_ADP3338
- removed UCT2, UCT3: AP2111H-3.3TRG1, Package_TO_SOT_SMD:SOT-223, symbol Sheet1-altium-import:root_0_ADP3338
- removed X3: 302-S101, Library:302-S101, symbol Sheet1-altium-import:root_0_HEADER_5X2
- added AX3: SJ1-3523N, Library:ST-222_1, symbol Sheet1-altium-import:root_0_mirrored_ST-222
- added C10, C2, C3, C4, C5, C8: 100nF, Capacitor_SMD:C_0603_1608Metric, symbol Sheet1-altium-import:root_1_C_0805
- added C103, C105, C15, C18, C203, C22, C23, C29, C36: 4.7uF, Capacitor_SMD:C_0603_1608Metric, symbol Sheet1-altium-import:root_0_C_0805
- added J2: 10067847-001RLF, Library:AMPHENOL_10067847-001RLF, symbol Library:10067847-001RLF
- added MP1: M2.5 x 1.5mm, Library:WA-SMSI_9774015151, symbol Library:WA-SMSI_9774XXX151
- added R1, R11, R2, R36: 10k, Resistor_SMD:R_0603_1608Metric, symbol Sheet1-altium-import:root_2_R_0805
- added R10, R20, R21, R22, R23, R24, R25, R7, R8, R9: 100E, Resistor_SMD:R_0603_1608Metric, symbol Sheet1-altium-import:root_2_R_0805
- added R13: 300k, Resistor_SMD:R_0603_1608Metric, symbol Sheet1-altium-import:root_2_R_0805
- added R14, R15, R16, R17, R18, R19, R3, R4, R5, R6: 200E, Resistor_SMD:R_0603_1608Metric, symbol Sheet1-altium-import:root_2_R_0805
- added R26, R35: 1k, Resistor_SMD:R_0603_1608Metric, symbol Sheet1-altium-import:root_1_R_0805
- added R27, R28, R29, R30, R31, R32, R33, R34: 75E, Resistor_SMD:R_0603_1608Metric, symbol Sheet1-altium-import:root_2_R_0805
- added S1: EVQ-P7A01P, Library:SW_EVQ-P7A01P, symbol Library:EVQ-P7A01P
- added S2: PTS526SM20SMTR21_LFS, Library:PTS526SM20SMTR21LFS, symbol Library:PTS526SM20SMTR21_LFS
- added U1: SOM_FPGA_LP, Library:SOM_FPGA_LP, symbol Library:SOM_FPGA_LP
- added U4: MAX3814, Package_QFP:TQFP-32_5x5mm_P0.5mm, symbol Library:MAX3814
- added U6: ESP32-S3-WROOM-1-N8R8, Library:MODULE_ESP32-S3-WROOM-1-N8R8, symbol Library:ESP32-S3-WROOM-1-N8R8
- added VR1: AP7366EA-33W5-7, Library:SOT-25-AP7366EA, symbol Library:AP7366EA-33W5-7
- added X2: SS-53000-001, Library:STEWART_SS-53000-001, symbol Library:SS-53000-001
- added X3: 490107671012_JTAG, Library:490107671012, symbol Library:490107671012
- C30: value 100nF -> 4.7uF; DIGIKEY 311-1088-1-ND -> 1276-2087-1-ND; LCSC (none) -> C107368
Connections:
- net +2V5: now also U14.10 (OE), U14.2 (VCCA); no longer C13.1, C14.1, C21.1
- net +3.3V: now also C11.1, C12.2, C13.2, C14.2, C19.2, C37.2, C36.2, R1.2, R2.2, R36.1, U1.9 (+3V3), U4.29 (LEVEL), U4.32 (VCC), U4.4 (VCC), U4.5 (VCC), U4.9 (VCC), U6.2 (3V3); no longer C30.2, C7.1
- net +3.3VDAC: now also C105.2, C22.2, VR1.2 (GND), VR1.5 (OUT)
- net +3V3: now also C21.2, C15.2, C23.2, J2.4 (VDD); no longer C9.2, U14.10 (OE), U14.2 (VCCA)
- net +5V: now also C20.1, C30.2, C44.1, C7.1, U1.1 (+5V), U1.3 (+5V), U1.5 (+5V), U1.7 (+5V), VR1.1 (IN), X2.18 (SUPPLY_+5V)
- net ADC_BCK: now also U1.44 (B3-IO2P)
- net ADC_DOUT: now also U1.50 (B3-IO6N)
- net ADC_LRCK: now also U1.46 (B3-IO2N)
- net ADC_SCKI: now also U1.48 (B3-IO6P)
- net DAC_BCK: now also U1.54 (B3-IO10N), U1.66 (B4-IO2N)
- net DAC_DIN: now also U1.64 (B4-IO2P)
- net DAC_FLT: now also U1.58 (B3-IO11N)
- net DAC_LRCK: now also U1.62 (B3-IO13N)
- net DAC_SCK: now also U1.52 (B3-IO10P), U1.56 (B3-IO11P)
- net DAC_XSMT: now also U1.60 (B3-IO13P)
- net GND: now also C12.1, C13.1, C14.1, C21.1, C37.1, C38.1, AX3.1, AX3.M (Mount), C15.1, C22.1, C23.1, C36.1, J2.3 (VSS), J2.6 (VSS__1), J2.G1 (GND), J2.G2 (GND__1), MP1.1, R11.1, R13.1, S1.2, S2.1 (COM_1), S2.2 (COM_2), S2.3 (NO_1), U1.121 (SHIELD), U1.122 (SHIELD), U1.123 (SHIELD), U1.124 (SHIELD), U1.2 (GND), U1.4 (GND), U1.6 (GND), U1.8 (GND), U4.12 (~{ENABLE}), U4.13 (VEE), U4.16 (VEE), U4.20 (VEE), U4.21 (VEE), U4.25 (VEE), U4.28 (VEE), U6.1 (GND), U6.40 (GND), U6.41 (GND), VR1.3 (EN), X2.11 (CLOCK_SHIELD), X2.17 (SUPPLY+GND), X2.2 (DATA2_SHIELD), X2.5 (DATA1_SHIELD), X2.8 (DATA0_SHIELD), X2.S1 (SHIELD), X2.S2 (SHIELD), X2.S3 (SHIELD), X2.S4 (SHIELD), X3.10 (GND), X3.2 (GND); no longer C12.2, C13.2, C14.2, C21.2, C37.2, C38.2, C6.1, C9.1
- net GNDA: now also C105.1, C29.1
- net HDDLED: now also U1.112 (B6-IO10)
- net SLTSOUND: now also C18.1
- net SLT_CLC: now also U1.25 (B2-CLK2)
- net SLT_MUX: now also U2.1 (G1), U2.19 (G2), U1.31 (B3-IO3); no longer U8.1 (G1), U8.19 (G2)
- net SLT_X0: now also U1.47 (B3-IO4-COP)
- net SLT_X1: now also U1.45 (B3-IO17)
- net SLT_X2: now also U1.43 (B3-IO16)
- net SLT_X3: now also U1.41 (B3-IO9)
- net SLT_X4: now also U1.39 (B3-IO8)
- net SLT_X5: now also U1.37 (B3-IO7)
- net SLT_X6: now also U1.35 (B3-IO12)
- net SLT_X7: now also U1.33 (B3-IO14)
- net SLT_Y0: now also U1.63 (B4-CLK13)
- net SLT_Y1: now also U1.61 (B4-IO8)
- net SLT_Y2: now also U1.59 (B4-IO1)
- net SLT_Y3: now also U1.57 (B4-IO5)
- net SLT_Y4: now also U1.55 (B3-CLK14)
- net SLT_Y5: now also U1.53 (B3-CLK15)
- net SLT_Y6: now also U1.51 (B3-IO15)
- net SLT_Y7: now also U1.49 (B3-IO4-CON)
- net TCK: now also U1.12 (TCK), X3.1 (TCK)
- net TDI: now also U1.10 (TDI), X3.9 (TDI)
- net TDO: now also U1.16 (TDO), X3.3 (TDO)
- net TMS: now also U1.14 (TMS), X3.5 (TMS)
- net ~{SLT_BUSDIR}: now also U1.19 (B2-IO6)
- net ~{SLT_INT}: now also U1.21 (B2-IO4)
- net ~{SLT_MUX}: now also U8.1 (G1), U8.19 (G2); no longer U2.1 (G1), U2.19 (G2)
- net ~{SLT_RESET}: now also U1.38 (B2-IO9P)
- net ~{SLT_RFSH}: now also U1.29 (B2-IO8)
- net ~{SLT_SLTSL}: now also U1.27 (B2-IO7)
- net ~{SLT_WAIT}: now also U1.23 (B2-CLK3)
- net at R103.2: now also C103.2
- net at AX2.4, AX2.5: now also C103.1
- net at R203.2: now also C203.2
- net at C35.2, R55.1, U9.3 (VCC): now also C29.2
- net at AX2.2, AX2.3: now also C203.1
- removed net +1V2: C11.1, C19.2, C20.1, C6.2
- new net: R14.1, R20.1
- new net: J2.8 (DAT1), R32.2
- new net: C3.2, U4.31 (INA-)
- new net: C8.2, U4.7 (INC-)
- new net: C18.2, R15.1, R20.2, R21.1
- new net: R17.1, R22.2, R23.1
- new net: AX3.4, AX3.5, R26.2
- new net: C5.2, U4.3 (INB-)
- new net: C10.2, U4.11 (IND-)
- new net: C4.2, U4.2 (INB+)
- new net: J2.2 (CMD), R30.2
- new net: C2.2, U4.30 (INA+)
- new net: AX3.2, AX3.3, R35.2
- new net: R18.1, R23.2, R24.1
- new net: J2.5 (CLK), R29.2
- new net: R19.1, R24.2, R25.1
- new net: J2.WP, R27.2
- new net: C6.2, U4.6 (INC+)
- new net: R16.1, R21.2, R22.1
- new net: J2.9 (DAT2), R33.2
- new net: J2.7 (DAT0), R31.2
- new net: J2.1 (DAT3/CD), R34.2
- new net: J2.CD, R28.2
- new net: C9.2, U4.10 (IND+)
- new net +IO1V8: U1.113 (+1V8), U1.115 (+1V8)
- new net +IO2V5: U1.109 (+2V5), U1.111 (+2V5), U1.114 (VCCB2)
- new net +IO3V3: U1.116 (VCCB3), U1.117 (+3V3), U1.118 (VCCB4), U1.119 (+3V3), U1.120 (VCCB5)
- new net DBG_RXD: R35.1
- new net DBG_TXD: R26.1
- new net ESP_BOOT_MODE: S2.4 (NO_2), U6.27 (IO0/BOOT)
- new net ESP_EN: R11.2, U6.3 (EN)
- new net ESP_IO1: U6.39 (IO1)
- new net ESP_IO10: U6.18 (IO10)
- new net ESP_IO11: U6.19 (IO11)
- new net ESP_IO12: U6.20 (IO12)
- new net ESP_IO13: U6.21 (IO13)
- new net ESP_IO14: U6.22 (IO14)
- new net ESP_IO15: U6.8 (IO15)
- new net ESP_IO16: U6.9 (IO16)
- new net ESP_IO17: U6.10 (IO17)
- new net ESP_IO18: U6.11 (IO18)
- new net ESP_IO2: U6.38 (IO2)
- new net ESP_IO21: U6.23 (IO21)
- new net ESP_IO3: U6.15 (IO3)
- new net ESP_IO35: U6.28 (IO35)
- new net ESP_IO36: U6.29 (IO36)
- new net ESP_IO37: U6.30 (IO37)
- new net ESP_IO38: U6.31 (IO38)
- new net ESP_IO39: U6.32 (IO39)
- new net ESP_IO4: U6.4 (IO4)
- new net ESP_IO40: U6.33 (IO40)
- new net ESP_IO41: U6.34 (IO41)
- new net ESP_IO42: U6.35 (IO42)
- new net ESP_IO45: U6.26 (IO45)
- new net ESP_IO46: U6.16 (IO46)
- new net ESP_IO47: U6.24 (IO47)
- new net ESP_IO48: U6.25 (IO48)
- new net ESP_IO5: U6.5 (IO5)
- new net ESP_IO6: U6.6 (IO6)
- new net ESP_IO7: U6.7 (IO7)
- new net ESP_IO8: U6.12 (IO8)
- new net ESP_IO9: U6.17 (IO9)
- new net ESP_RXD: U6.36 (RXD0)
- new net ESP_TXD: U6.37 (TXD0)
- new net HDMI_A+: R3.2, U4.27 (OUTA+), X2.1 (DATA2+)
- new net HDMI_A-: R3.1, U4.26 (OUTA-), X2.3 (DATA2-)
- new net HDMI_B+: R4.2, U4.23 (OUTB+), X2.4 (DATA1+)
- new net HDMI_B-: R4.1, U4.22 (OUTB-), X2.6 (DATA1-)
- new net HDMI_C+: R5.2, U4.19 (OUTC+), X2.7 (DATA0+)
- new net HDMI_C-: R5.1, U4.18 (OUTC-), X2.9 (DATA0-)
- new net HDMI_D+: R6.2, U4.15 (OUTD+), X2.10 (CLOCK+)
- new net HDMI_D-: R6.1, U4.14 (OUTD-), X2.12 (CLOCK-)
- new net HDMI_SCL: R1.1, U1.42 (B3-IO1N), X2.15 (SCL)
- new net HDMI_SDA: R2.1, U1.40 (B3-IO1P), X2.16 (SDA)
- new net JTAGVCC: U1.18 (+2V5), X3.4 (VCC)
- new net LVDS_CLK_N: C10.1, R10.1, U1.32 (B2-IO5N)
- new net LVDS_CLK_P: C9.1, R10.2, U1.34 (B2-IO5P)
- new net LVDS_D0_N: C8.1, R9.1, U1.28 (B2-IO3N)
- new net LVDS_D0_P: C6.1, R9.2, U1.30 (B2-IO3P)
- new net LVDS_D1_N: C5.1, R8.1, U1.24 (B2-IO2N)
- new net LVDS_D1_P: C4.1, R8.2, U1.26 (B2-IO2P)
- new net LVDS_D2_N: C3.1, R7.1, U1.20 (B2-IO1N)
- new net LVDS_D2_P: C2.1, R7.2, U1.22 (B2-IO1P)
- new net PUSH_BUTTON: C38.2, R36.2, S1.1, U1.110 (B6-IO1N)
- new net SD_CD: R28.1, U1.82 (B4-IO10N)
- new net SD_CLK: R29.1, U1.68 (B4-IO3P)
- new net SD_CMD: R30.1, U1.70 (B4-IO3N)
- new net SD_DAT0: R31.1, U1.72 (B4-IO4P)
- new net SD_DAT1: R32.1, U1.74 (B4-IO4N)
- new net SD_DAT2: R33.1, U1.76 (B4-IO7P)
- new net SD_DAT3: R13.2, R34.1, U1.78 (B4-IO7N)
- new net SD_WP: R27.1, U1.80 (B4-IO10P)
- new net SND0: R19.2, U1.83 (B5-IO5)
- new net SND1: R18.2, U1.81 (B5-CLK7)
- new net SND2: R17.2, U1.79 (B5-CLK6)
- new net SND3: R16.2, U1.77 (B5-IO2)
- new net SND4: R15.2, U1.75 (B5-IO1)
- new net SND5: R14.2, U1.73 (B5-IO6)
- no-connect marks 0 -> 4
Other:
- note added: "Analog Power"
- note added: "Button"
- note added: "Debug terminal"
- note added: "HDMI Output"
- note added: "SD-Card"
- note added: "SLT_MUX = 0 (Data and control)"
- note added: "SLT_MUX = 1 (Address)"
- note added: "WiFi / Bluetooth / Co-processor"
- note removed: "Altera Cyclone 10LP"
- note removed: "EEPROM"
- note removed: "JTAG"
- note removed: "Power"
- moved on the sheet: AX2, C11, C16, C17, C19, C20, C28, C31, C32, C33, C34, C35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

Commit message: Schematic work in progress
Parts:
- removed AX3: SJ1-3523N, Library:ST-222_1, symbol Sheet1-altium-import:root_0_mirrored_ST-222
- removed C1, C205: 10uF 10V, Capacitor_Tantalum_SMD:CP_EIA-3216-10_Kemet-I_Pad1.58x1.35mm_HandSolder, symbol Sheet1-altium-import:root_0_CAP100RP
- removed C101, C201: 2.2nF, Capacitor_SMD:C_0603_1608Metric, symbol Sheet1-altium-import:root_1_C_0805
- removed C102, C24, C25, C27, C31, C32, C33, C34, C35: 100nF, Capacitor_SMD:C_0603_1608Metric, symbol Sheet1-altium-import:root_1_C_0805
- removed C104, C204: 2.2uF, Capacitor_SMD:C_0603_1608Metric, symbol Sheet1-altium-import:root_0_C_0805
- removed C203, C29, C30: 4.7uF, Capacitor_SMD:C_0603_1608Metric, symbol Sheet1-altium-import:root_0_C_0805
- removed C26: 10uF 10V, Capacitor_Tantalum_SMD:CP_EIA-3216-10_Kemet-I_Pad1.58x1.35mm_HandSolder, symbol Sheet1-altium-import:root_3_CAP100RP
- removed C28: 10uF 10V, Capacitor_Tantalum_SMD:CP_EIA-3216-10_Kemet-I_Pad1.58x1.35mm_HandSolder, symbol Sheet1-altium-import:root_2_CAP100RP
- removed R103, R203: 75E, Resistor_SMD:R_0603_1608Metric, symbol Sheet1-altium-import:root_2_R_0805
- removed R104, R204: 470E, Resistor_SMD:R_0603_1608Metric, symbol Sheet1-altium-import:root_2_R_0805
- removed R26, R35: 1k, Resistor_SMD:R_0603_1608Metric, symbol Sheet1-altium-import:root_1_R_0805
- removed R55: 220E, Resistor_SMD:R_0603_1608Metric, symbol Sheet1-altium-import:root_0_R_0805
- removed R64: 10E, Resistor_SMD:R_0603_1608Metric, symbol Sheet1-altium-import:root_2_R_0805
- removed S2: PTS526SM20SMTR21_LFS, Library:PTS526SM20SMTR21LFS, symbol Library:PTS526SM20SMTR21_LFS
- removed U5: PCM5101APWR, Package_SO:TSSOP-20_4.4x6.5mm_P0.65mm, symbol Library:PCM510xA
- removed U9: PCM1808PWR, Package_SO:TSSOP-14_4.4x5mm_P0.65mm, symbol Library:PCM1808
- added C1, C25, C28, C29, C39, C40: 4.7uF, Capacitor_SMD:C_0603_1608Metric, symbol Device:C_Small
- added C24, C26, C31, C32, C42, C43, C46, C47: 100nF, Capacitor_SMD:C_0603_1608Metric, symbol Device:C_Small
- added C27, C30, C33, C34, C35, C41, C48, C49, C50, C51: 1uF, Capacitor_SMD:C_0603_1608Metric, symbol Device:C_Small
- added J3, J4: UJ20-C-H-G-SMT-2-P16-TR, Library:SAMESKY_UJ20-C-H-G-SMT-2-P16-TR, symbol Library:UJ20-C-H-G-SMT-2-P16-TR
- added J5: Conn_01x08, Connector_PinHeader_2.00mm:PinHeader_1x08_P2.00mm_Vertical, symbol Connector_Generic:Conn_01x08
- added J6: Conn_01x06, Connector_PinHeader_2.00mm:PinHeader_1x06_P2.00mm_Vertical, symbol Connector_Generic:Conn_01x06
- added J7: Conn_02x04_Odd_Even, Connector_PinHeader_2.00mm:PinHeader_2x04_P2.00mm_Vertical, symbol Connector_Generic:Conn_02x04_Odd_Even
- added Q1, Q2: UM6K34NTCN, Package_TO_SOT_SMD:SOT-363_SC-70-6, symbol Library:Q_Dual_NMOS_UM6K34NTCN
- added R12, R26, R35, R37, R38, R39, R40, R41, R50: 10k, Resistor_SMD:R_0603_1608Metric, symbol Device:R_Small
- added R42: 100E, Resistor_SMD:R_0603_1608Metric, symbol Device:R_Small
- added R43, R44: 1k, Resistor_SMD:R_0603_1608Metric, symbol Device:R_Small
- added R46, R47, R48, R49: 5k1, Resistor_SMD:R_0603_1608Metric, symbol Device:R_Small
- added S3: EVQ-P7A01P, Library:SW_EVQ-P7A01P, symbol Library:EVQ-P7A01P
- added U11, U13: TPD1E05U06DPY, Package_SON:Texas_DPY0002A_0.6x1mm_P0.65mm, symbol Power_Protection:TPD1E05U06DPY
- added U5: NAU88C22A, Library:QFN-32-NAU88C22YG, symbol Library:NAU88C22A
- added U7: MCP2221AT-I/SL, Package_SO:SOIC-14_3.9x8.7mm_P1.27mm, symbol Library:MCP2221AT-I_SL
- added U9: AP22816AKEWT, Package_TO_SOT_SMD:SOT-23-5, symbol Power_Management:AP22816AKEWT
- AX1, AX2: symbol Sheet1-altium-import:root_0_mirrored_ST-222 -> Library:ST-222
- C10, C11, C12, C13, C14, C16, C17, C19, C2, C20, C21, C3, C37, C38, C4, C44, C45, C5, C6, C8, C9: symbol Sheet1-altium-import:root_1_C_0805 -> Device:C_Small
- C103: value 4.7uF -> 1uF; symbol Sheet1-altium-import:root_0_C_0805 -> Device:C_Small; DIGIKEY 1276-2087-1-ND -> 4988-NMC0603X7R105K6.3TRPFCT-ND; LCSC C107368 -> (none)
- C105, C15, C18, C22, C23, C36, C7: symbol Sheet1-altium-import:root_0_C_0805 -> Device:C_Small
- LED1: symbol Sheet1-altium-import:root_2_LED -> Device:LED
- R1, R10, R11, R13, R14, R15, R16, R17, R18, R19, R2, R20, R21, R22, R23, R24, R27, R28, R29, R3, R30, R31, R32, R33, R34, R36, R4, R5, R6, R7, R8, R9, R99: symbol Sheet1-altium-import:root_2_R_0805 -> Device:R_Small
- R25: value 100E -> 200E; symbol Sheet1-altium-import:root_2_R_0805 -> Device:R_Small; DIGIKEY 4463-TFAS0603R1000F-T5CT-ND -> 4463-TFAS0603R2000F-T5CT-ND
- R45: symbol Sheet1-altium-import:root_0_R_0805 -> Device:R_Small
- R72: symbol Sheet1-altium-import:root_1_R_0805 -> Device:R_Small
- U10: symbol 74xGxx:74LVC1GU04 -> Library:74LVC1GU04
- X1: symbol Sheet1-altium-import:root_0_EDGE50/MSX -> Library:EDGE50-MSX
Connections:
- net +2V5 is gone; now on net +IO2V5: U14.10 (OE), U14.2 (VCCA)
- net DAC_DIN is gone; now on net SD_CLK: U1.64 (B4-IO2P)
- net ESP_IO17 is gone; now on net ESP_IO17/SCL: U6.10 (IO17)
- net ESP_IO18 is gone; now on net ESP_IO18/SDA: U6.11 (IO18)
- net ESP_IO21 is gone; now on net ESP_IO21/USBEN: U6.23 (IO21)
- net ESP_IO35 is gone; now on net ESP_IO35/GP0: U6.28 (IO35)
- net ESP_IO36 is gone; now on net ESP_IO36/GP1: U6.29 (IO36)
- net ESP_IO37 is gone; now on net ESP_IO37/GP2: U6.30 (IO37)
- net ESP_IO38 is gone; now on net ESP_IO38/GP3: U6.31 (IO38)
- net +3V3: now also C11.2, C12.1, C13.1, C14.1, C16.2, C17.2, C19.1, C36.2, C37.1, C45.2, LED1.2 (A), R1.2, R2.2, R36.1, U1.11 (+3V3), U1.13 (+3V3), U1.15 (+3V3), U1.9 (+3V3), U4.29 (LEVEL), U4.32 (VCC), U4.4 (VCC), U4.5 (VCC), U4.9 (VCC), U6.2 (3V3), C24.2, C41.2, C46.2, R26.1, R37.2, R38.2, R41.2, U5.14 (VDDB), U7.1 (VDD), U7.11 (VUSB); no longer C16.1, C17.1, C45.1
- net +5V: now also C20.2, C44.2, VR1.3 (EN), C1.2, C27.2, C30.1, C32.1, C43.2, C47.2, U9.5 (IN); no longer C20.1, C44.1
- net +IO1V8: now also C40.2, U5.13 (VDDC)
- net +IO2V5: now also C42.2
- net DBG_RXD: now also U1.65 (B4-CLK12), U7.5 (URx)
- net DBG_TXD: now also U1.67 (B4-IO9), U7.6 (UTx)
- net ESP_BOOT_MODE: now also U1.87 (B5-IO10), C31.1, R26.2, S3.1
- net ESP_EN: now also U1.85 (B5-IO11)
- net ESP_IO1: now also U1.89 (B6-IO2)
- net ESP_IO10: now also U1.107 (B6-IO9)
- net ESP_IO11: now also U1.102 (B5-IO8N)
- net ESP_IO12: now also U1.104 (B5-IO9P)
- net ESP_IO13: now also U1.106 (B5-IO9N)
- net ESP_IO14: now also U1.108 (B6-IO1P)
- net ESP_IO15: now also U1.110 (B6-IO1N)
- net ESP_IO16: now also U1.112 (B6-IO10)
- net ESP_IO2: now also U1.91 (B6-IO6)
- net ESP_IO3: now also U1.93 (B6-IO3)
- net ESP_IO39: now also U1.100 (eB5-IO8P)
- net ESP_IO4: now also U1.95 (B6-IO4)
- net ESP_IO40: now also J7.5 (Pin_5)
- net ESP_IO41: now also J7.6 (Pin_6)
- net ESP_IO42: now also J7.7 (Pin_7)
- net ESP_IO45: now also J7.1 (Pin_1)
- net ESP_IO46: now also J7.2 (Pin_2)
- net ESP_IO47: now also J7.3 (Pin_3)
- net ESP_IO48: now also J7.4 (Pin_4)
- net ESP_IO5: now also U1.97 (B6-CLK5)
- net ESP_IO6: now also U1.99 (B6-CLK4)
- net ESP_IO7: now also U1.101 (B6-IO8)
- net ESP_IO8: now also U1.103 (B6-IO7)
- net ESP_IO9: now also U1.105 (B6-IO5)
- net ESP_RXD: now also U1.82 (B4-IO10N)
- net ESP_TXD: now also U1.80 (B4-IO10P)
- net GND: now also C105.1, C11.1, C12.2, C13.2, C14.2, C16.1, C17.1, C19.2, C20.1, C37.2, C38.2, C44.1, C45.1, R25.2, R72.1, C1.1, C24.1, C25.1, C26.1, C27.1, C30.2, C31.2, C32.2, C39.1, C41.1, C42.1, C43.1, C46.1, C47.1, J3.A1_B12 (GND), J3.B1_A12 (GND__1), J3.SH1 (SHIELD), J3.SH2 (SHIELD__1), J3.SH3 (SHIELD__2), J3.SH4 (SHIELD__3), J4.A1_B12 (GND), J4.B1_A12 (GND__1), J4.SH1 (SHIELD), J4.SH2 (SHIELD__1), J4.SH3 (SHIELD__2), J4.SH4 (SHIELD__3), J7.8 (Pin_8), Q1.1 (S), Q1.4 (S), Q2.1 (S), R12.1, R40.1, R46.1, R47.1, R48.1, R49.1, R50.2, S3.2, U11.2 (GND), U13.2 (GND), U5.24 (VSSSPK), U5.28 (VSSA), U5.33 (EXP), U7.14 (VSS), U9.2 (GND); no longer C11.2, C12.1, C13.1, C14.1, C16.2, C17.2, C19.1, C20.2, C23.1, C37.1, C38.1, C44.2, C45.2, R72.2, VR1.3 (EN)
- net GNDA: now also C23.1, C28.2, C29.2, C40.1, J5.7 (Pin_7), J5.8 (Pin_8), J6.5 (Pin_5), J6.6 (Pin_6), R35.2, R39.2, U5.12 (VSSD); no longer C105.1
- net HDDLED: now also R45.1, U1.36 (B2-IO9N); no longer LED1.1 (K), U1.112 (B6-IO10)
- net HDMI_A+: no longer R3.2
- net HDMI_A-: now also R3.2; no longer R3.1, U4.26 (OUTA-)
- net HDMI_B+: no longer R4.2
- net HDMI_B-: now also R4.2; no longer R4.1, U4.22 (OUTB-)
- net HDMI_C+: no longer R5.2
- net HDMI_C-: now also R5.2; no longer R5.1, U4.18 (OUTC-)
- net HDMI_D+: no longer R6.2
- net HDMI_D-: now also R6.2; no longer R6.1, U4.14 (OUTD-)
- net LVDS_CLK_N: no longer C10.1
- net LVDS_CLK_P: now also C9.2; no longer C9.1, R10.2
- net LVDS_D0_N: no longer C8.1
- net LVDS_D0_P: now also C6.2; no longer C6.1, R9.2
- net LVDS_D1_N: no longer C5.1
- net LVDS_D1_P: now also C4.2; no longer C4.1, R8.2
- net LVDS_D2_N: no longer C3.1
- net LVDS_D2_P: now also C2.2; no longer C2.1, R7.2
- net PUSH_BUTTON: now also C38.1, U1.71 (B4-IO11); no longer C38.2, U1.110 (B6-IO1N)
- net SD_CD: now also U1.78 (B4-IO7N); no longer U1.82 (B4-IO10N)
- net SD_CLK: no longer U1.68 (B4-IO3P)
- net SD_CMD: now also U1.66 (B4-IO2N); no longer U1.70 (B4-IO3N)
- net SD_DAT0: now also U1.68 (B4-IO3P); no longer U1.72 (B4-IO4P)
- net SD_DAT1: now also U1.70 (B4-IO3N); no longer U1.74 (B4-IO4N)
- net SD_DAT2: now also U1.72 (B4-IO4P); no longer U1.76 (B4-IO7P)
- net SD_DAT3: now also U1.74 (B4-IO4N); no longer U1.78 (B4-IO7N)
- net SD_WP: now also U1.76 (B4-IO7P); no longer U1.80 (B4-IO10P)
- net ~{SLT_WAIT}: now also R72.2; no longer R72.1
- net at R45.2: now also LED1.1 (K); no longer LED1.2 (A)
- net at U4.31 (INA-): now also C3.1; no longer C3.2
- net at U4.7 (INC-): now also C8.1; no longer C8.2
- net at U4.3 (INB-): now also C5.1; no longer C5.2
- net at U4.11 (IND-): now also C10.1; no longer C10.2
- net at AX2.2, AX2.3: now also C33.2
- net at U4.2 (INB+): now also C4.1; no longer C4.2
- net at U4.30 (INA+): now also C2.1; no longer C2.2
- net at AX2.4, AX2.5: now also C103.2; no longer C103.1
- net at AX1.2, AX1.3: now also C35.1, R39.1
- net at AX1.4, AX1.5: now also C34.1, R35.1
- net ESP_USB_Dn: now reaches U6.13 (IO19/USB_Dn)
- net ESP_USB_Dn: now also J3.A7 (DN1), J3.B7 (DN2)
- net ESP_USB_Dp: now reaches U6.14 (IO20/USB-Dp)
- net ESP_USB_Dp: now also J3.A6 (DP1), J3.B6 (DP2)
- net at U4.6 (INC+): now also C6.1; no longer C6.2
- net ~{DBG_ACT}: now reaches U1.69 (B4-IO6)
- net ~{DBG_ACT}: now also Q1.5 (G), Q1.6 (D), R37.1
- net HDMI_CEC: now reaches U1.84 (B4-IO12-COP)
- net HDMI_CEC: now also R42.1
- net HDMI_HPD: now reaches U1.86 (B4-IO12-CON)
- net HDMI_HPD: now also Q2.6 (D), R41.1
- net ESP_IO17/SCL: now reaches U1.88 (B5-IO4P)
- net ESP_IO17/SCL: now also U7.10 (SCL)
- net ESP_IO18/SDA: now reaches U1.90 (B5-IO4N)
- net ESP_IO18/SDA: now also U7.9 (SDA)
- net ESP_IO35/GP0: now reaches U1.92 (B5-IO3P)
- net ESP_IO35/GP0: now also R43.2
- net ESP_IO36/GP1: now reaches U1.94 (B5-IO3N)
- net ESP_IO36/GP1: now also R44.2
- net ESP_IO37/GP2: now reaches U1.96 (B5-IO7P)
- net ESP_IO37/GP2: now also U7.7 (GP2)
- net ESP_IO38/GP3: now reaches U1.98 (B5-IO7N)
- net ESP_IO38/GP3: now also U7.8 (GP3)
- net CEC: now reaches X2.13 (CEC)
- net CEC: now also R42.2, U13.1 (I/O)
- net HPD: now reaches X2.19 (HPD)
- net HPD: now also Q2.2 (G), R40.2, U11.1 (I/O)
- net at U4.10 (IND+): now also C9.1; no longer C9.2
- removed net +3.3V: C11.1, C12.2, C13.2, C14.2, C19.2, C36.2, C37.2, R1.2, R2.2, R36.1, R45.1, U1.9 (+3V3), U4.29 (LEVEL), U4.32 (VCC), U4.4 (VCC), U4.5 (VCC), U4.9 (VCC), U6.2 (3V3)
- net +3.3VDAC renamed +3V3DAC
- net +3V3DAC: now also C39.2, U5.26 (VDDSPK), U5.31 (VDDA)
- net ADC_BCK renamed CODEC_MCK
- net CODEC_MCK: now also U5.11 (MCLK)
- net ADC_DOUT renamed CODEC_DACIN
- net CODEC_DACIN: now also U5.10 (DACIN)
- net ADC_LRCK renamed CODEC_BCK
- net CODEC_BCK: now also U5.8 (BCLK)
- net ADC_SCKI renamed CODEC_FS
- net CODEC_FS: now also U5.7 (FS)
- net DAC_BCK renamed CODEC_SCLK
- net CODEC_SCLK: now also U5.16 (SCLK); no longer U1.66 (B4-IO2N)
- net DAC_FLT renamed CODEC_CSB
- net CODEC_CSB: now also U5.15 (CSB/GPIO1)
- net DAC_LRCK renamed ESP_IO21/USBEN
- net ESP_IO21/USBEN: now also R50.1, U9.4 (EN)
- net DAC_SCK renamed CODEC_ADCOUT
- net CODEC_ADCOUT: now also U5.9 (ADCOUT); no longer U1.56 (B3-IO11P)
- net DAC_XSMT renamed CODEC_MODE
- net CODEC_MODE: now also U5.18 (MODE)
- new net: C3.2, R7.2
- new net: C8.2, R9.2
- new net: C5.2, R8.2
- new net: R44.1, U7.3 (GP1)
- new net: C10.2, R10.2
- new net: C103.1, U5.19 (LAUXIN)
- new net: J4.A5 (CC1), R46.2
- new net: J4.B5 (CC2), R47.2
- new net: J5.1 (Pin_1), U5.3 (LLIN/GPIO2)
- new net: J5.2 (Pin_2), U5.6 (RLIN/GPIO3)
- new net: C48.2, J5.3 (Pin_3)
- new net: C49.2, J5.4 (Pin_4)
- new net: C50.2, J5.5 (Pin_5)
- new net: C51.2, J5.6 (Pin_6)
- new net: J3.A5 (CC1), R48.2
- new net: J3.B5 (CC2), R49.2
- new net: C33.1, U5.20 (RAUXIN)
- new net: C51.1, U5.4 (RMICP)
- new net: R5.1, U4.18 (OUTC-)
- new net: R3.1, U4.26 (OUTA-)
- new net: C35.2, U5.22 (AUXOUT2)
- new net: C34.2, U5.21 (AUXOUT1)
- new net: C28.1, U5.27 (VREF)
- new net: C29.1, U5.32 (MICBIAS)
- new net: R6.1, U4.14 (OUTD-)
- new net: C49.1, U5.1 (LMICP)
- new net: C48.1, U5.2 (LMICN)
- new net: J6.3 (Pin_3), U5.23 (RSPKOUT)
- new net: J6.4 (Pin_4), U5.25 (LSPKOUT)
- new net: J6.2 (Pin_2), U5.29 (RHP)
- new net: J6.1 (Pin_1), U5.30 (LHP)
- new net: C50.1, U5.5 (RMICN)
- new net: R4.1, U4.22 (OUTB-)
- new net: R43.1, U7.2 (GP0)
- new net CODEC_SDIO: U1.56 (B3-IO11P), U5.17 (SDIO)
- new net DBG_Dn: J4.A7 (DN1), J4.B7 (DN2), U7.12 (D-)
- new net DBG_Dp: J4.A6 (DP1), J4.B6 (DP2), U7.13 (D+)
- new net DBG_VBUS: J4.A4_B9 (VBUS), J4.B4_A9 (VBUS__1), Q1.2 (G), R12.2
- new net USB_VBUS: C25.2, C26.2, J3.A4_B9 (VBUS), J3.B4_A9 (VBUS__1), U9.1 (OUT)
- new net ~{USB_RST}: Q1.3 (D), R38.1, U7.4 (~{RST})
- no-connect marks 4 -> 23
Other:
- note added: "WiFi / Audio / USB /Co-processor"
- note removed: "WiFi / Bluetooth / Co-processor"
- moved on the sheet: AX1, AX2, J1, J2, MP1, S1, U1, U10, U12, U14, U2, U3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
