File: board/HyperFusionXC.kicad_sch (KiCad schematic)
At the start: 140 parts, among them J1 Conn_01x02_Pin, J2 10067847-001RLF, J3 UJ20-C-H-G-SMT-2-P16-TR, J4 UJ20-C-H-G-SMT-2-P16-TR, J5 Conn_01x08, J6 Conn_01x06, J7 Conn_02x04_Odd_Even, Q1 UM6K34NTCN, Q2 UM6K34NTCN, U1 SOM_FPGA_LP, U10 SN74LVC1G04DCKR, U11 TPD1E05U06DPY, U12 TXS0108EPWR, U13 TPD1E05U06DPY, U14 TXS0108EPWR, U2 74AHC541, U3 74AHC541, U4 MAX3814, U5 NAU88C22A, U6 ESP32-S3-WROOM-1-N8R8, U7 MCP2221AT-I/SL, U8 74AHC541, U9 AP22816AKEWT, X1 EDGE50/MSX, X2 SS-53000-001, X3 490107671012_JTAG

Commit message: Schematic work in progress
Parts:
- removed J6: Conn_01x06, Connector_PinHeader_2.00mm:PinHeader_1x06_P2.00mm_Vertical, symbol Connector_Generic:Conn_01x06
- removed J7: Conn_02x04_Odd_Even, Connector_PinHeader_2.00mm:PinHeader_2x04_P2.00mm_Vertical, symbol Connector_Generic:Conn_02x04_Odd_Even
- removed Q2: UM6K34NTCN, Package_TO_SOT_SMD:SOT-363_SC-70-6, symbol Library:Q_Dual_NMOS_UM6K34NTCN
- removed R41: 10k, Resistor_SMD:R_0603_1608Metric, symbol Device:R_Small
- removed R42: 100E, Resistor_SMD:R_0603_1608Metric, symbol Device:R_Small
- removed U11, U13: TPD1E05U06DPY, Package_SON:Texas_DPY0002A_0.6x1mm_P0.65mm, symbol Power_Protection:TPD1E05U06DPY
- removed U9: AP22816AKEWT, Package_TO_SOT_SMD:SOT-23-5, symbol Power_Management:AP22816AKEWT
- added C52: 1uF, Capacitor_SMD:C_0603_1608Metric, symbol Device:C_Small
- added C53: 100nF, Capacitor_SMD:C_0603_1608Metric, symbol Device:C_Small
- added C54: 4.7uF, Capacitor_SMD:C_0603_1608Metric, symbol Device:C_Small
- added J6: Conn_01x05, Connector_PinSocket_2.00mm:PinSocket_1x05_P2.00mm_Vertical, symbol Connector_Generic:Conn_01x05
- added J7: Conn_02x05_Odd_Even, Connector_PinHeader_2.00mm:PinHeader_2x05_P2.00mm_Vertical, symbol Connector_Generic:Conn_02x05_Odd_Even
- added U11, U9: AP22816BKAWT-7, Package_TO_SOT_SMD:SOT-23-5, symbol Library:AP22816BKAWT
- added U15: TXB0104D, Package_SO:SOIC-14_3.9x8.7mm_P1.27mm, symbol Logic_LevelTranslator:TXB0104D
- R40: value 10k -> 1k; DIGIKEY RMCF0603FT10K0CT-ND -> RMCF0603FT1K00CT-ND
Connections:
- net +3V3: now also R50.2, J7.2 (Pin_2), U15.1 (VCCA), U15.8 (OE); no longer R1.2, R2.2
- net +5V: now also C52.2, U11.4 (IN), U15.14 (VCCB), U9.4 (IN); no longer X2.18 (SUPPLY_+5V)
- net CODEC_ADCOUT: now also U1.69 (B4-IO6); no longer U1.52 (B3-IO10P)
- net CODEC_BCK: now also U1.67 (B4-IO9); no longer U1.46 (B3-IO2N)
- net CODEC_DACIN: now also U1.71 (B4-IO11); no longer U1.50 (B3-IO6N)
- net CODEC_FS: now also U1.61 (B4-IO8); no longer U1.48 (B3-IO6P)
- net CODEC_MCK: now also U1.62 (B3-IO13N); no longer U1.44 (B3-IO2P)
- net CODEC_MODE: now also U1.66 (B4-IO2N); no longer U1.60 (B3-IO13P)
- net CODEC_SCLK: now also U1.60 (B3-IO13P); no longer U1.54 (B3-IO10N)
- net CODEC_SDIO: now also U1.64 (B4-IO2P); no longer U1.56 (B3-IO11P)
- net DBG_RXD: now also U1.78 (B4-IO7N); no longer U1.65 (B4-CLK12)
- net DBG_TXD: now also U1.76 (B4-IO7P); no longer U1.67 (B4-IO9)
- net ESP_BOOT_MODE: now also U1.88 (B5-IO4P); no longer U1.87 (B5-IO10)
- net ESP_EN: now also U1.82 (B4-IO10N); no longer U1.85 (B5-IO11)
- net ESP_IO10: now also J7.3 (Pin_3)
- net ESP_IO11: now also J7.5 (Pin_5)
- net ESP_IO12: now also J7.7 (Pin_7)
- net ESP_IO13: now also J7.4 (Pin_4)
- net ESP_IO14: now also J7.6 (Pin_6)
- net ESP_IO15: now also J7.8 (Pin_8)
- net ESP_IO16: now also J7.10 (Pin_10)
- net ESP_IO17/SCL: now also U1.90 (B5-IO4N); no longer U1.88 (B5-IO4P)
- net ESP_IO18/SDA: now also U1.92 (B5-IO3P); no longer U1.90 (B5-IO4N)
- net ESP_IO21/USBEN: now also U1.86 (B4-IO12-CON), U9.1 (~{EN}); no longer U1.62 (B3-IO13N)
- net ESP_IO35/GP0: now also U1.94 (B5-IO3N); no longer U1.92 (B5-IO3P)
- net ESP_IO36/GP1: now also U1.96 (B5-IO7P); no longer U1.94 (B5-IO3N)
- net ESP_IO37/GP2: now also U1.98 (B5-IO7N); no longer U1.96 (B5-IO7P)
- net ESP_IO38/GP3: now also U1.100 (B5-IO8P); no longer U1.98 (B5-IO7N)
- net ESP_IO9: now also J7.1 (Pin_1)
- net ESP_RXD: now also U1.84 (B4-IO12-COP); no longer U1.82 (B4-IO10N)
- net ESP_TXD: now also U1.79 (B5-CLK6); no longer U1.80 (B4-IO10P)
- net GND: now also R40.2, C52.1, C53.1, C54.1, J7.9 (Pin_9), U11.2 (GND), U15.7 (GND), U9.2 (GND); no longer R40.1, R50.2, U4.12 (~{ENABLE})
- net GNDA: now also J5.1 (Pin_1), J6.1 (Pin_1); no longer J5.7 (Pin_7)
- net HDMI_A+: now also R3.2
- net HDMI_A-: now also R3.1, U4.26 (OUTA-); no longer R3.2
- net HDMI_B+: now also R4.2
- net HDMI_B-: now also R4.1, U4.22 (OUTB-); no longer R4.2
- net HDMI_C+: now also R5.2
- net HDMI_C-: now also R5.1, U4.18 (OUTC-); no longer R5.2
- net HDMI_CEC: now also U1.72 (B4-IO4P), U15.2 (A1); no longer U1.84 (B4-IO12-COP)
- net HDMI_D+: now also R6.2
- net HDMI_D-: now also R6.1, U4.14 (OUTD-); no longer R6.2
- net HDMI_HPD: now also U1.74 (B4-IO4N), U15.5 (A4); no longer U1.86 (B4-IO12-CON)
- net HDMI_SCL: now also U1.70 (B4-IO3N), U15.3 (A2); no longer R1.1, U1.42 (B3-IO1N), X2.15 (SCL)
- net HDMI_SDA: now also U1.68 (B4-IO3P), U15.4 (A3); no longer R2.1, U1.40 (B3-IO1P), X2.16 (SDA)
- net LVDS_CLK_N: now also C10.2
- net LVDS_CLK_P: now also R10.2
- net LVDS_D0_N: now also C8.2
- net LVDS_D0_P: now also R9.2
- net LVDS_D1_N: now also C5.2
- net LVDS_D1_P: now also R8.2
- net LVDS_D2_N: now also C3.2
- net LVDS_D2_P: now also R7.2
- net PUSH_BUTTON: now also U1.81 (B5-CLK7); no longer U1.71 (B4-IO11)
- net SD_CD: now also U1.46 (B3-IO2N); no longer U1.78 (B4-IO7N)
- net SD_CLK: now also U1.48 (B3-IO6P); no longer U1.64 (B4-IO2P)
- net SD_CMD: now also U1.44 (B3-IO2P); no longer U1.66 (B4-IO2N)
- net SD_DAT0: now also U1.50 (B3-IO6N); no longer U1.68 (B4-IO3P)
- net SD_DAT1: now also U1.52 (B3-IO10P); no longer U1.70 (B4-IO3N)
- net SD_DAT2: now also U1.42 (B3-IO1N); no longer U1.72 (B4-IO4P)
- net SD_DAT3: now also U1.40 (B3-IO1P); no longer U1.74 (B4-IO4N)
- net SD_WP: now also U1.54 (B3-IO10N); no longer U1.76 (B4-IO7P)
- net SLT_Y0: now also U1.65 (B4-CLK12); no longer U1.63 (B4-CLK13)
- net SLT_Y1: now also U1.63 (B4-CLK13); no longer U1.61 (B4-IO8)
- net SND0: now also U1.87 (B5-IO10); no longer U1.83 (B5-IO5)
- net SND1: now also U1.85 (B5-IO11); no longer U1.81 (B5-CLK7)
- net SND2: now also U1.83 (B5-IO5); no longer U1.79 (B5-CLK6)
- net USB_VBUS: now also U9.5 (OUT)
- net ~{SLT_RFSH}: now also U1.23 (B2-CLK3); no longer U1.29 (B2-IO8)
- net ~{SLT_WAIT}: now also U1.29 (B2-IO8); no longer U1.23 (B2-CLK3)
- net at U5.3 (LLIN/GPIO2): now also J5.4 (Pin_4); no longer J5.1 (Pin_1)
- net at J5.2 (Pin_2): now also C49.2; no longer U5.6 (RLIN/GPIO3)
- net at J5.5 (Pin_5): now also C51.2; no longer C50.2
- net at J5.6 (Pin_6): now also C50.2; no longer C51.2
- net at U5.23 (RSPKOUT): now also J6.4 (Pin_4)
- net at U5.25 (LSPKOUT): now also J6.5 (Pin_5)
- net at U5.29 (RHP): now also J6.3 (Pin_3)
- net at U5.30 (LHP): now also J6.2 (Pin_2)
- net CEC: no longer names the net of X2.13 (CEC)
- net CEC: now also U15.13 (B1)
- net ESP_IO39: no longer names the net of U6.32 (IO39)
- net ESP_IO39: no longer U1.100 (eB5-IO8P)
- net ESP_IO40: no longer names the net of U6.33 (IO40)
- net ESP_IO41: no longer names the net of U6.34 (IO41)
- net ESP_IO42: no longer names the net of U6.35 (IO42)
- net ESP_IO45: no longer names the net of U6.26 (IO45)
- net ESP_IO46: no longer names the net of U6.16 (IO46)
- net ESP_IO47: no longer names the net of U6.24 (IO47)
- net ESP_IO48: no longer names the net of U6.25 (IO48)
- net HPD: no longer names the net of X2.19 (HPD)
- net HPD: now also R40.1, U15.10 (B4); no longer R40.2
- net ~{DBG_ACT}: no longer names the net of Q1.5 (G), Q1.6 (D), R37.1
- net ~{DBG_ACT}: no longer U1.69 (B4-IO6)
- net ~{USB_RST} renamed ~{DBG_RST}
- net ~{DBG_RST}: now also U1.80 (B4-IO10P)
- new net: C53.2, C54.2, R1.1, R2.1, U11.5 (OUT), X2.18 (SUPPLY_+5V)
- new net: R1.2, U15.12 (B2), X2.15 (SCL)
- new net: J5.7 (Pin_7), U5.6 (RLIN/GPIO3)
- new net: R2.2, U15.11 (B3), X2.16 (SDA)
- new net ~{HDMI_EN}: U1.56 (B3-IO11P), U11.1 (~{EN}), U4.12 (~{ENABLE})
- no-connect marks 23 -> 29
Other:
- note added: "2V5"
- moved on the sheet: C10, C11, C12, C13, C14, C19, C2, C20, C25, C26, C27, C3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

Commit message: PCB work in progress
Parts:
- added FL1: DLM0NSN900HY2D, Library:FIL_DLM0NSN900HY2D, symbol Filter:Choke_CommonMode_FerriteCore_1243
Connections:
- net CODEC_MODE: now also U1.68 (B4-IO3P); no longer U1.66 (B4-IO2N)
- net DBG_RXD: now also U1.80 (B4-IO10P); no longer U1.78 (B4-IO7N)
- net DBG_TXD: now also U1.79 (B5-CLK6); no longer U1.76 (B4-IO7P)
- net ESP_BOOT_MODE: now also U1.66 (B4-IO2N); no longer U1.88 (B5-IO4P)
- net ESP_EN: now also U1.112 (B6-IO10); no longer U1.82 (B4-IO10N)
- net ESP_IO1: now also U1.96 (B5-IO7P); no longer U1.89 (B6-IO2)
- net ESP_IO10: now also U1.108 (B6-IO1P); no longer U1.107 (B6-IO9)
- net ESP_IO11: now also U1.106 (B5-IO9N); no longer U1.102 (B5-IO8N)
- net ESP_IO13: now also U1.102 (B5-IO8N); no longer U1.106 (B5-IO9N)
- net ESP_IO14: now also U1.100 (B5-IO8P); no longer U1.108 (B6-IO1P)
- net ESP_IO15: now also U1.101 (B6-IO8); no longer U1.110 (B6-IO1N)
- net ESP_IO16: now also U1.89 (B6-IO2); no longer U1.112 (B6-IO10)
- net ESP_IO17/SCL: now also U1.107 (B6-IO9); no longer U1.90 (B5-IO4N)
- net ESP_IO18/SDA: now also U1.105 (B6-IO5); no longer U1.92 (B5-IO3P)
- net ESP_IO2: now also U1.94 (B5-IO3N); no longer U1.91 (B6-IO6)
- net ESP_IO21/USBEN: now also U1.98 (B5-IO7N); no longer U1.86 (B4-IO12-CON)
- net ESP_IO3: now also U1.91 (B6-IO6); no longer U1.93 (B6-IO3)
- net ESP_IO35/GP0: now also U1.82 (B4-IO10N); no longer U1.94 (B5-IO3N)
- net ESP_IO36/GP1: now also U1.84 (B4-IO12-COP); no longer U1.96 (B5-IO7P)
- net ESP_IO37/GP2: now also U1.86 (B4-IO12-CON); no longer U1.98 (B5-IO7N)
- net ESP_IO38/GP3: now also U1.88 (B5-IO4P); no longer U1.100 (B5-IO8P)
- net ESP_IO4: now also U1.93 (B6-IO3); no longer U1.95 (B6-IO4)
- net ESP_IO5: now also U1.95 (B6-IO4); no longer U1.97 (B6-CLK5)
- net ESP_IO6: now also U1.97 (B6-CLK5); no longer U1.99 (B6-CLK4)
- net ESP_IO7: now also U1.99 (B6-CLK4); no longer U1.101 (B6-IO8)
- net ESP_IO9: now also U1.110 (B6-IO1N); no longer U1.105 (B6-IO5)
- net ESP_RXD: now also U1.90 (B5-IO4N); no longer U1.84 (B4-IO12-COP)
- net ESP_TXD: now also U1.92 (B5-IO3P); no longer U1.79 (B5-CLK6)
- net ESP_USB_Dn: now also FL1.2; no longer J3.A7 (DN1), J3.B7 (DN2)
- net ESP_USB_Dp: now also FL1.3; no longer J3.A6 (DP1), J3.B6 (DP2)
- net HDMI_CEC: now also U1.70 (B4-IO3N), U15.5 (A4); no longer U1.72 (B4-IO4P), U15.2 (A1)
- net HDMI_HPD: now also U1.76 (B4-IO7P), U15.2 (A1); no longer U1.74 (B4-IO4N), U15.5 (A4)
- net HDMI_SCL: now also U1.72 (B4-IO4P), U15.4 (A3); no longer U1.70 (B4-IO3N), U15.3 (A2)
- net HDMI_SDA: now also U1.74 (B4-IO4N), U15.3 (A2); no longer U1.68 (B4-IO3P), U15.4 (A3)
- net ~{DBG_RST}: now also U1.78 (B4-IO7N); no longer U1.80 (B4-IO10P)
- net at R1.2, U15.12 (B2): now also X2.16 (SDA); no longer X2.15 (SCL)
- net at R40.1, X2.19 (HPD): now also U15.13 (B1); no longer U15.10 (B4)
- net at R2.2, U15.11 (B3): now also X2.15 (SCL); no longer X2.16 (SDA)
- net at X2.13 (CEC): now also U15.10 (B4); no longer U15.13 (B1)
- new net: FL1.4, J3.A6 (DP1), J3.B6 (DP2)
- new net: FL1.1, J3.A7 (DN1), J3.B7 (DN2)
Other:
- moved on the sheet: C25, C26, C27, C31, C36, C37, C41, J3, J7, R11, R26, R48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

Commit message: PCB work in progress
Parts:
- added FL2: DLM0NSN900HY2D, Library:FIL_DLM0NSN900HY2D, symbol Filter:Choke_CommonMode_FerriteCore_1243
Connections:
- net DBG_Dn: now also FL2.2; no longer J4.A7 (DN1), J4.B7 (DN2)
- net DBG_Dp: now also FL2.3; no longer J4.A6 (DP1), J4.B6 (DP2)
- net ESP_IO1: now also J7.4 (Pin_4)
- net ESP_IO10: now also J7.7 (Pin_7); no longer J7.3 (Pin_3)
- net ESP_IO11: now also J7.8 (Pin_8); no longer J7.5 (Pin_5)
- net ESP_IO12: now also J7.5 (Pin_5); no longer J7.7 (Pin_7)
- net ESP_IO13: now also J7.6 (Pin_6); no longer J7.4 (Pin_4)
- net ESP_IO14: now also J7.3 (Pin_3); no longer J7.6 (Pin_6)
- net ESP_IO15: no longer J7.8 (Pin_8)
- net ESP_IO16: no longer J7.10 (Pin_10)
- net ESP_IO2: now also J7.1 (Pin_1)
- net ESP_IO9: now also J7.10 (Pin_10); no longer J7.1 (Pin_1)
- new net: FL2.4, J4.A6 (DP1), J4.B6 (DP2)
- new net: FL2.1, J4.A7 (DN1), J4.B7 (DN2)
Changed lines of the file:
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@@
 	)
 	(junction
-		(at 527.05 54.61)
-		(diameter 0)
-		(color 0 0 0 0)
-	)
-	(junction
 		(at 368.3 181.61)
 		(diameter 0)
@@
 	)
 	(junction
+		(at 527.05 54.61)
+		(diameter 0)
+		(color 0 0 0 0)
+	)
+	(junction
 		(at 226.06 39.37)
 		(diameter 0)
@@
 	)
 	(junction
-		(at 508 173.99)
+		(at 525.78 59.69)
 		(diameter 0)
 		(color 0 0 0 0)
 	)
 	(junction
-		(at 246.38 72.39)
+		(at 508 173.99)
 		(diameter 0)
 		(color 0 0 0 0)
 	)
 	(junction
-		(at 525.78 57.15)
+		(at 246.38 72.39)
 		(diameter 0)
 		(color 0 0 0 0)
@@
 	(wire
 		(pts
+			(xy 524.51 59.69) (xy 525.78 59.69)
+		)
+		(stroke
+			(width 0)
+			(type default)
+		)
+	)
+	(wire
+		(pts
 			(xy 525.78 95.25) (xy 528.32 95.25)
 		)
@@
 	(wire
 		(pts
-			(xy 514.35 57.15) (xy 525.78 57.15)
+			(xy 502.92 59.69) (xy 514.35 59.69)
 		)
 		(stroke
@@
 	(wire
 		(pts
-			(xy 514.35 54.61) (xy 527.05 54.61)
+			(xy 502.92 54.61) (xy 514.35 54.61)
 		)
 		(stroke
@@
 	(wire
 		(pts
+			(xy 524.51 54.61) (xy 527.05 54.61)
+		)
+		(stroke
+			(width 0)
+			(type default)
+		)
+	)
+	(wire
+		(pts
 			(xy 123.19 72.39) (xy 171.45 72.39)
 		)
@@
 	(wire
 		(pts
+			(xy 525.78 59.69) (xy 525.78 57.15)
+		)
+		(stroke
+			(width 0)
+			(type default)
+		)
+	)
+	(wire
+		(pts
 			(xy 378.46 156.21) (xy 384.81 156.21)
 		)
@@
 	(wire
 		(pts
-			(xy 525.78 64.77) (xy 525.78 57.15)
+			(xy 525.78 64.77) (xy 525.78 59.69)
 		)
 		(stroke
@@
 		)
 	)
-	(label "ESP_IO12"
+	(label "ESP_IO10"
 		(at 369.57 259.08 0)
 		(effects
@@
 		)
 	)
-	(label "ESP_IO15"
+	(label "ESP_IO11"
 		(at 405.13 259.08 180)
 		(effects
@@
 		)
 	)
-	(label "ESP_IO11"
+	(label "ESP_IO12"
 		(at 369.57 256.54 0)
 		(effects
@@
 	)
 	(label "DBG_Dn"
-		(at 514.35 54.61 0)
+		(at 502.92 54.61 0)
 		(effects
 			(font
@@
 		)
 	)
-	(label "ESP_IO13"
+	(label "ESP_IO1"
 		(at 405.13 254 180)
 		(effects
@@
 		)
 	)
-	(label "ESP_IO16"
+	(label "ESP_IO9"
 		(at 405.13 261.62 180)
 		(effects
@@
 		)
 	)
-	(label "ESP_IO9"
+	(label "ESP_IO2"
 		(at 369.57 251.46 0)
 		(effects
@@
 		)
 	)
-	(label "ESP_IO10"
+	(label "ESP_IO14"
 		(at 369.57 254 0)
 		(effects
@@
 	)
 	(label "DBG_Dp"
-		(at 514.35 57.15 0)
+		(at 502.92 59.69 0)
 		(effects
 			(font
@@
 		)
 	)
-	(label "ESP_IO14"
+	(label "ESP_IO13"
 		(at 405.13 256.54 180)
 		(effects
@@
 					(unit 1)
 				)
+			)
+		)
+	)
+	(symbol
+		(lib_id "Filter:Choke_CommonMode_FerriteCore_1243")
+		(at 519.43 57.15 0)
+		(mirror y)
+		(unit 1)
+		(exclude_from_sim no)
+		(in_bom yes)
+		(on_board yes)
+		(dnp no)
+		(property "Reference" "FL2"
+			(at 519.938 52.832 0)
+			(effects
+				(font
+					(size 1.27 1.27)
+				)
+			)
+		)
+		(property "Value" "DLM0NSN900HY2D"
+			(at 515.874 61.976 0)
+			(effects
+				(font
+					(size 1.27 1.27)
+				)
+			)
+		)
+		(property "Footprint" "Library:FIL_DLM0NSN900HY2D"
+			(at 519.43 63.5 0)
+			(effects
+				(font
+					(size 1.27 1.27)
+				)
+				(hide yes)
+			)
+		)
+		(property "Datasheet" "~"
+			(at 519.43 65.405 0)
+			(effects
+				(font
+					(size 1.27 1.27)
+				)
+				(hide yes)
+			)
+		)
+		(property "Description" "Generic common-mode choke, ferrite core, 1243 pin order"
+			(at 515.366 57.912 0)
+			(effects
+				(font
+					(size 1.27 1.27)
+				)
+				(hide yes)
+			)
+		)
+		(property "DIGIKEY" "490-DLM0NSN900HY2DCT-ND"
+			(at 519.43 57.15 0)
+			(effects
+				(font
+					(size 1.27 1.27)
+				)
+				(hide yes)
+			)
+		)
+		(pin "1"
+		)
+		(pin "4"
+		)
+		(pin "3"
+		)
+		(pin "2"
+		)
+		(instances
+			(project "HyperFusionXC"
+				(path "/dc7b2672-e830-4a16-8d9e-d44ab4cff2d4"
+					(reference "FL2")
+					(unit 1)
+				)

Commit message: PCB work in progress
Parts:
- removed J1: Conn_01x02_Pin, Library:JUMPER_1, symbol Connector:Conn_01x02_Pin
- added J1: Conn_01x03, Connector_PinHeader_2.54mm:PinHeader_1x03_P2.54mm_Vertical, symbol Connector_Generic:Conn_01x03
Connections:
- net +3V3: now also J1.3 (Pin_3)
- net +5V: now also J1.2 (Pin_2)
- net GND: now also J1.1 (Pin_1)
Changed lines of the file:
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@@
 	(wire
 		(pts
-			(xy 36.83 236.22) (xy 50.8 236.22)
-		)
-		(stroke
-			(width 0)
-			(type default)
-		)
-	)
-	(wire
-		(pts
 			(xy 242.57 48.26) (xy 234.95 48.26)
 		)
@@
 	(wire
 		(pts
+			(xy 30.48 233.68) (xy 30.48 241.3)
+		)
+		(stroke
+			(width 0)
+			(type default)
+		)
+	)
+	(wire
+		(pts
 			(xy 115.57 88.9) (xy 115.57 81.28)
 		)
@@
 	(wire
 		(pts
+			(xy 30.48 241.3) (xy 46.99 241.3)
+		)
+		(stroke
+			(width 0)
+			(type default)
+		)
+	)
+	(wire
+		(pts
 			(xy 132.08 59.69) (xy 140.97 59.69)
 		)
@@
 	(wire
 		(pts
+			(xy 35.56 238.76) (xy 46.99 238.76)
+		)
+		(stroke
+			(width 0)
+			(type default)
+		)
+	)
+	(wire
+		(pts
 			(xy 318.77 185.42) (xy 300.99 185.42)
 		)
@@
 	(wire
 		(pts
-			(xy 33.02 237.49) (xy 33.02 243.84)
-		)
-		(stroke
-			(width 0)
-			(type default)
-		)
-	)
-	(wire
-		(pts
 			(xy 439.42 199.39) (xy 450.85 199.39)
 		)
@@
 	(wire
 		(pts
+			(xy 40.64 229.87) (xy 46.99 229.87)
+		)
+		(stroke
+			(width 0)
+			(type default)
+		)
+	)
+	(wire
+		(pts
 			(xy 389.89 186.69) (xy 397.51 186.69)
 		)
@@
 	(wire
 		(pts
-			(xy 41.91 243.84) (xy 41.91 238.76)
-		)
-		(stroke
-			(width 0)
-			(type default)
-		)
-	)
-	(wire
-		(pts
 			(xy 234.95 48.26) (xy 234.95 52.07)
 		)
@@
 	(wire
 		(pts
+			(xy 46.99 229.87) (xy 46.99 236.22)
+		)
+		(stroke
+			(width 0)
+			(type default)
+		)
+	)
+	(wire
+		(pts
 			(xy 242.57 302.26) (xy 260.35 302.26)
 		)
@@
 	(wire
 		(pts
+			(xy 35.56 233.68) (xy 35.56 238.76)
+		)
+		(stroke
+			(width 0)
+			(type default)
+		)
+	)
+	(wire
+		(pts
 			(xy 199.39 356.87) (xy 189.23 356.87)
 		)
@@
 	(wire
 		(pts
-			(xy 33.02 243.84) (xy 41.91 243.84)
-		)
-		(stroke
-			(width 0)
-			(type default)
-		)
-	)
-	(wire
-		(pts
 			(xy 370.84 323.85) (xy 370.84 334.01)
 		)
@@
 	(wire
 		(pts
-			(xy 41.91 238.76) (xy 50.8 238.76)
-		)
-		(stroke
-			(width 0)
-			(type default)
-		)
-	)
-	(wire
-		(pts
 			(xy 318.77 210.82) (xy 300.99 210.82)
 		)
@@
 	(symbol
 		(lib_id "power:GND")
-		(at 36.83 236.22 0)
+		(at 40.64 229.87 0)
 		(unit 1)
 		(exclude_from_sim no)
@@
 		(fields_autoplaced yes)
 		(property "Reference" "#PWR043"
-			(at 36.83 242.57 0)
+			(at 40.64 236.22 0)
 			(effects
 				(font
@@
 		)
 		(property "Value" "GND"
-			(at 36.83 241.3 0)
+			(at 40.64 234.95 0)
 			(effects
 				(font
@@
 		)
 		(property "Footprint" ""
-			(at 36.83 236.22 0)
+			(at 40.64 229.87 0)
 			(effects
 				(font
@@
 		)
 		(property "Datasheet" ""
-			(at 36.83 236.22 0)
+			(at 40.64 229.87 0)
 			(effects
 				(font
@@
 		)
 		(property "Description" "Power symbol creates a global label with name \"GND\" , ground"
-			(at 36.83 236.22 0)
+			(at 40.64 229.87 0)
 			(effects
 				(font
@@
 	(symbol
 		(lib_id "power:+5V")
-		(at 33.02 237.49 0)
+		(at 35.56 233.68 0)
 		(unit 1)
 		(exclude_from_sim no)
@@
 		(fields_autoplaced yes)
 		(property "Reference" "#PWR051"
-			(at 33.02 241.3 0)
+			(at 35.56 237.49 0)
 			(effects
 				(font
@@
 		)
 		(property "Value" "+5V"
-			(at 33.02 232.41 0)
+			(at 35.56 228.6 0)
 			(effects
 				(font
@@
 		)
 		(property "Footprint" ""
-			(at 33.02 237.49 0)
+			(at 35.56 233.68 0)
 			(effects
 				(font
@@
 		)
 		(property "Datasheet" ""
-			(at 33.02 237.49 0)
+			(at 35.56 233.68 0)
 			(effects
 				(font
@@
 		)
 		(property "Description" "Power symbol creates a global label with name \"+5V\""
-			(at 33.02 237.49 0)
+			(at 35.56 233.68 0)
 			(effects
 				(font
@@
 	)
 	(symbol
-		(lib_id "Connector:Conn_01x02_Pin")
-		(at 55.88 236.22 0)
-		(mirror y)
-		(unit 1)
-		(exclude_from_sim no)
-		(in_bom yes)
-		(on_board yes)
-		(dnp no)
-		(property "Reference" "J1"
-			(at 55.245 231.14 0)
-			(effects
-				(font
-					(size 1.27 1.27)
-				)
-			)
-		)
-		(property "Value" "Conn_01x02_Pin"
-			(at 55.245 233.68 0)
-			(effects
-				(font
-					(size 1.27 1.27)
-				)
-			)
-		)
-		(property "Footprint" "Library:JUMPER_1"
-			(at 55.88 236.22 0)
-			(effects
-				(font
-					(size 1.27 1.27)
-				)
-				(hide yes)
-			)
-		)
-		(property "Datasheet" "~"
-			(at 55.88 236.22 0)
-			(effects
-				(font
-					(size 1.27 1.27)
-				)
-				(hide yes)
-			)
-		)
-		(property "Description" ""
-			(at 55.88 236.22 0)
-			(effects
-				(font
-					(size 1.27 1.27)
-				)
-			)
-		)
-		(pin "2"
-		)
-		(pin "1"
-		)
-		(instances
-			(project "Carnivore2"
-				(path "/dc7b2672-e830-4a16-8d9e-d44ab4cff2d4"
-					(reference "J1")
-					(unit 1)
-				)
-			)
-		)
-	)
-	(symbol
 		(lib_id "power:GND")
 		(at 106.68 156.21 0)
@@
 	)
 	(symbol
+		(lib_id "Connector_Generic:Conn_01x03")
+		(at 52.07 238.76 0)
+		(unit 1)
+		(exclude_from_sim no)
+		(in_bom yes)
+		(on_board yes)
+		(dnp no)
+		(fields_autoplaced yes)
+		(property "Reference" "J1"
+			(at 54.61 237.4899 0)
+			(effects
+				(font
+					(size 1.27 1.27)
+				)
+				(justify left)
+			)
+		)
+		(property "Value" "Conn_01x03"
+			(at 54.61 240.0299 0)
+			(effects
+				(font
+					(size 1.27 1.27)
+				)
+				(justify left)
+			)
+		)
+		(property "Footprint" "Connector_PinHeader_2.54mm:PinHeader_1x03_P2.54mm_Vertical"
+			(at 52.07 238.76 0)
+			(effects
+				(font
+					(size 1.27 1.27)
+				)
+				(hide yes)
+			)
+		)
+		(property "Datasheet" "~"
+			(at 52.07 238.76 0)
+			(effects
+				(font
+					(size 1.27 1.27)
+				)
+				(hide yes)
+			)
+		)
+		(property "Description" "Generic connector, single row, 01x03, script generated (kicad-library-utils/schlib/autogen/connector/)"
+			(at 52.07 238.76 0)
+			(effects
+				(font
+					(size 1.27 1.27)
+				)
+				(hide yes)
+			)
+		)
+		(pin "1"
+		)
+		(pin "2"
+		)
+		(pin "3"
+		)
+		(instances
+			(project ""
+				(path "/dc7b2672-e830-4a16-8d9e-d44ab4cff2d4"
+					(reference "J1")
+					(unit 1)
+				)
+			)
+		)
+	)
+	(symbol
 		(lib_id "74xx:74AHC541")
 		(at 176.53 359.41 0)
@@
 					(unit 1)
 				)
+			)
+		)
+	)
+	(symbol
+		(lib_id "power:+3V3")
+		(at 30.48 233.68 0)
+		(unit 1)
+		(exclude_from_sim no)
+		(in_bom yes)
+		(on_board yes)
+		(dnp no)
+		(fields_autoplaced yes)
+		(property "Reference" "#PWR096"
+			(at 30.48 237.49 0)
+			(effects
+				(font
+					(size 1.27 1.27)
+				)
+				(hide yes)
+			)
+		)
+		(property "Value" "+3V3"
+			(at 30.48 228.6 0)
+			(effects
+				(font
+					(size 1.27 1.27)
+				)
+			)
+		)
+		(property "Footprint" ""
+			(at 30.48 233.68 0)
+			(effects
+				(font
+					(size 1.27 1.27)
+				)
+				(hide yes)
+			)
+		)
+		(property "Datasheet" ""
+			(at 30.48 233.68 0)
+			(effects
+				(font
+					(size 1.27 1.27)
+				)
+				(hide yes)
+			)
+		)
+		(property "Description" "Power symbol creates a global label with name \"+3V3\""
+			(at 30.48 233.68 0)
+			(effects
+				(font
+					(size 1.27 1.27)
+				)
+				(hide yes)
+			)
+		)
+		(pin "1"
+		)
+		(instances
+			(project "HyperFusionXC"
+				(path "/dc7b2672-e830-4a16-8d9e-d44ab4cff2d4"
+					(reference "#PWR096")
+					(unit 1)
+				)
